File: KiCad/Generic3.kicad_pcb (KiCad board)
At the start: 2 copper layers, 35 x 21.5 mm, 38 parts, among them J1 DC, J2 I/O, J3 USB-C, U1 ESP32-PICO-MINI-02, U2 FT231XQ, U3 LMR16006+FB, U4 QR

Commit message: Tidy
Changed lines of the file:
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@@
       (effects (font (size 1 1) (thickness 0.15)))
+    )
+    (fp_text user "${DATE}" (at 0 -3.6 -90 unlocked) (layer "F.SilkS")
+      (effects (font (size 0.75 0.75) (thickness 0.1)))
+    )
+    (fp_text user "Max 2mm" (at -8.1 -8.4 unlocked) (layer "F.Fab")
+      (effects (font (size 0.5 0.5) (thickness 0.1)))
     )
     (fp_text user "ANTENNA" (at -3 -7.7 90) (layer "F.Fab")
       (effects (font (size 0.787402 0.787402) (thickness 0.15)))
     )
-    (fp_text user "From edge" (at -7.3 -8.4 unlocked) (layer "F.Fab")
+    (fp_text user "Min 5mm" (at 10.2 -8.2 unlocked) (layer "F.Fab")
       (effects (font (size 0.5 0.5) (thickness 0.1)))
     )
@@
       (effects (font (size 0.5 0.5) (thickness 0.1)))
     )
-    (fp_text user "Max 2mm" (at -8.1 -8.4 unlocked) (layer "F.Fab")
+    (fp_text user "From edge" (at -7.3 -8.4 unlocked) (layer "F.Fab")
       (effects (font (size 0.5 0.5) (thickness 0.1)))
     )
@@
       (effects (font (size 0.5 0.5) (thickness 0.1)))
     )
-    (fp_text user "Min 5mm" (at 10.2 -8.2 unlocked) (layer "F.Fab")
-      (effects (font (size 0.5 0.5) (thickness 0.1)))
-    )
     (fp_line (start 6.6 -11) (end -6.6 -11) (layer "F.CrtYd") (width 0.05))
+    (fp_line (start 6.6 5.6) (end 6.6 -11) (layer "F.CrtYd") (width 0.05))
+    (fp_line (start -6.6 -11) (end -6.6 5.6) (layer "F.CrtYd") (width 0.05))
     (fp_line (start -6.6 5.6) (end 6.6 5.6) (layer "F.CrtYd") (width 0.05))
-    (fp_line (start -6.6 -11) (end -6.6 5.6) (layer "F.CrtYd") (width 0.05))
-    (fp_line (start 6.6 5.6) (end 6.6 -11) (layer "F.CrtYd") (width 0.05))
+    (fp_line (start 11.6 -5.6) (end 6.6 -5.6) (layer "F.Fab") (width 0.1))
+    (fp_line (start -8.6 -5.6) (end -6.6 -5.6) (layer "F.Fab") (width 0.1))
+    (fp_line (start -8.6 -11) (end -8.6 -5.6) (layer "F.Fab") (width 0.1))
+    (fp_line (start -6.6 -5.6) (end 6.6 -5.6) (layer "F.Fab") (width 0.127))
+    (fp_line (start -6.6 -11) (end -8.6 -11) (layer "F.Fab") (width 0.1))
+    (fp_line (start 11.6 -12) (end 15.1 -12) (layer "F.Fab") (width 0.1))
+    (fp_line (start 6.6 -5.6) (end 6.6 5.6) (layer "F.Fab") (width 0.127))
+    (fp_line (start -6.6 -5.6) (end -6.6 -11) (layer "F.Fab") (width 0.127))
+    (fp_line (start -8.6 -12) (end -8.6 -11) (layer "F.Fab") (width 0.1))
+    (fp_line (start 11.6 -11) (end 11.6 -12) (layer "F.Fab") (width 0.1))
+    (fp_line (start -8.6 -5.6) (end -8.6 -2.3) (layer "F.Fab") (width 0.1))
+    (fp_line (start 6.6 -11) (end 6.6 -5.6) (layer "F.Fab") (width 0.127))
+    (fp_line (start 6.6 -11) (end 11.6 -11) (layer "F.Fab") (width 0.1))
+    (fp_line (start -6.6 5.6) (end -6.6 -5.6) (layer "F.Fab") (width 0.127))
+    (fp_line (start 6.6 5.6) (end -6.6 5.6) (layer "F.Fab") (width 0.127))
     (fp_line (start -6.6 -11) (end 6.6 -11) (layer "F.Fab") (width 0.127))
-    (fp_line (start -6.6 -11) (end -8.6 -11) (layer "F.Fab") (width 0.1))
-    (fp_line (start -8.6 -5.6) (end -8.6 -2.3) (layer "F.Fab") (width 0.1))
-    (fp_line (start 11.6 -12) (end 15.1 -12) (layer "F.Fab") (width 0.1))
-    (fp_line (start -6.6 -5.6) (end 6.6 -5.6) (layer "F.Fab") (width 0.127))
-    (fp_line (start 6.6 -11) (end 11.6 -11) (layer "F.Fab") (width 0.1))
-    (fp_line (start 11.6 -5.6) (end 6.6 -5.6) (layer "F.Fab") (width 0.1))
+    (fp_line (start 11.6 -11) (end 11.6 -5.6) (layer "F.Fab") (width 0.1))
     (fp_line (start 11.6 -12) (end -8.6 -12) (layer "F.Fab") (width 0.1))
-    (fp_line (start 6.6 5.6) (end -6.6 5.6) (layer "F.Fab") (width 0.127))
-    (fp_line (start 6.6 -11) (end 6.6 -5.6) (layer "F.Fab") (width 0.127))
-    (fp_line (start 6.6 -5.6) (end 6.6 5.6) (layer "F.Fab") (width 0.127))
-    (fp_line (start -8.6 -11) (end -8.6 -5.6) (layer "F.Fab") (width 0.1))
-    (fp_line (start -8.6 -5.6) (end -6.6 -5.6) (layer "F.Fab") (width 0.1))
-    (fp_line (start 11.6 -11) (end 11.6 -12) (layer "F.Fab") (width 0.1))
-    (fp_line (start -6.6 5.6) (end -6.6 -5.6) (layer "F.Fab") (width 0.127))
-    (fp_line (start 11.6 -11) (end 11.6 -5.6) (layer "F.Fab") (width 0.1))
-    (fp_line (start -8.6 -12) (end -8.6 -11) (layer "F.Fab") (width 0.1))
-    (fp_line (start -6.6 -5.6) (end -6.6 -11) (layer "F.Fab") (width 0.127))
     (pad "1" smd rect (at -5.9 -4 270) (size 0.8 0.4) (layers "F.Cu" "F.Paste" "F.Mask")
       (net 1 "GND") (pinfunction "GND") (pintype "power_in"))
@@
     (pad "48" smd rect (at -4.8 -4.9 270) (size 0.4 0.8) (layers "F.Cu" "F.Paste" "F.Mask")
       (net 1 "GND") (pinfunction "GND") (pintype "power_in"))
-    (pad "49" smd rect (at 1.975 0 270) (size 1.45 1.45) (layers "F.Cu" "F.Paste" "F.Mask")
-      (net 1 "GND") (pinfunction "GND") (pintype "power_in"))
-    (pad "49" smd rect (at 0 0 270) (size 1.45 1.45) (layers "F.Cu" "F.Paste" "F.Mask")
-      (net 1 "GND") (pinfunction "GND") (pintype "power_in"))
     (pad "49" smd roundrect (at -1.975 -1.975 270) (size 1.45 1.45) (layers "F.Cu" "F.Paste" "F.Mask") (roundrect_rratio 0)
       (chamfer_ratio 0.41) (chamfer top_left)
-      (net 1 "GND") (pinfunction "GND") (pintype "power_in"))
-    (pad "49" smd rect (at 1.975 -1.975 270) (size 1.45 1.45) (layers "F.Cu" "F.Paste" "F.Mask")
-      (net 1 "GND") (pinfunction "GND") (pintype "power_in"))
-    (pad "49" smd rect (at 0 1.975 270) (size 1.45 1.45) (layers "F.Cu" "F.Paste" "F.Mask")
       (net 1 "GND") (pinfunction "GND") (pintype "power_in"))
     (pad "49" smd rect (at -1.975 0 270) (size 1.45 1.45) (layers "F.Cu" "F.Paste" "F.Mask")
@@
     (pad "49" smd rect (at 1.975 1.975 270) (size 1.45 1.45) (layers "F.Cu" "F.Paste" "F.Mask")
       (net 1 "GND") (pinfunction "GND") (pintype "power_in"))
+    (pad "49" smd rect (at 1.975 0 270) (size 1.45 1.45) (layers "F.Cu" "F.Paste" "F.Mask")
+      (net 1 "GND") (pinfunction "GND") (pintype "power_in"))
     (pad "49" smd rect (at 0 -1.975 270) (size 1.45 1.45) (layers "F.Cu" "F.Paste" "F.Mask")
+      (net 1 "GND") (pinfunction "GND") (pintype "power_in"))
+    (pad "49" smd rect (at 1.975 -1.975 270) (size 1.45 1.45) (layers "F.Cu" "F.Paste" "F.Mask")
+      (net 1 "GND") (pinfunction "GND") (pintype "power_in"))
+    (pad "49" smd rect (at 0 1.975 270) (size 1.45 1.45) (layers "F.Cu" "F.Paste" "F.Mask")
+      (net 1 "GND") (pinfunction "GND") (pintype "power_in"))
+    (pad "49" smd rect (at 0 0 270) (size 1.45 1.45) (layers "F.Cu" "F.Paste" "F.Mask")
       (net 1 "GND") (pinfunction "GND") (pintype "power_in"))
     (pad "50" smd rect (at 5.95 -4.95 270) (size 0.7 0.7) (layers "F.Cu" "F.Paste" "F.Mask")
@@
     (pad "53" smd rect (at -5.95 -4.95 270) (size 0.7 0.7) (layers "F.Cu" "F.Paste" "F.Mask")
       (net 1 "GND") (pinfunction "GND") (pintype "power_in"))
-    (zone (net 0) (net_name "") (layers *.Cu) (hatch full 0.508)
+    (zone (net 0) (net_name "") (layer "F.Cu") (hatch full 0.508)
       (connect_pads (clearance 0))
       (min_thickness 0.01)
-      (keepout (tracks allowed) (vias not_allowed) (pads allowed ) (copperpour allowed) (footprints allowed))
+      (keepout (tracks not_allowed) (vias not_allowed) (pads not_allowed ) (copperpour not_allowed) (footprints allowed))
       (fill (thermal_gap 0.508) (thermal_bridge_width 0.508))
       (polygon
@@
       )
     )
-    (zone (net 0) (net_name "") (layer "F.Cu") (hatch full 0.508)
+    (zone (net 0) (net_name "") (layers *.Cu) (hatch full 0.508)
       (connect_pads (clearance 0))
       (min_thickness 0.01)
-      (keepout (tracks not_allowed) (vias not_allowed) (pads not_allowed ) (copperpour not_allowed) (footprints allowed))
+      (keepout (tracks allowed) (vias not_allowed) (pads allowed ) (copperpour allowed) (footprints allowed))
       (fill (thermal_gap 0.508) (thermal_bridge_width 0.508))
       (polygon

Commit message: Tidy
Parts:
- moved Logo1 0.49 mm to (167.1, 59.9)
Other:
- board text removed: "www.me.uk"
