File: KiCad/Generic3.kicad_sch (KiCad schematic)
At the start: 38 parts, among them J1 DC, J2 I/O, J3 USB-C, U1 ESP32-PICO-MINI-02, U2 FT231XQ, U3 LMR16006+FB, U4 QR

Commit message: Various minor tidy
Parts:
- J1: symbol Connector_Generic:Conn_01x02 -> RevK:PowerIn
- J3: symbol Connector:USB_C_Receptacle_USB2.0 -> RevK:USB-C
Connections:
- no-connect marks 12 -> 10
Changed lines of the file:
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@@
   (junction (at 179.07 40.64) (diameter 0) (color 0 0 0 0)
   )
-  (junction (at 170.815 43.18) (diameter 0) (color 0 0 0 0)
-  )
   (junction (at 184.785 63.5) (diameter 0) (color 0 0 0 0)
   )
@@
   (junction (at 180.975 31.75) (diameter 0) (color 0 0 0 0)
   )
-  (junction (at 170.815 40.64) (diameter 0) (color 0 0 0 0)
-  )
-  (no_connect (at 170.815 53.34))
   (no_connect (at 226.06 137.16))
-  (no_connect (at 170.815 55.88))
   (no_connect (at 46.99 80.01))
   (no_connect (at 46.99 72.39))
@@
     (stroke (width 0) (type default) (color 0 0 0 0))
   )
-  (wire (pts (xy 170.815 38.1) (xy 170.815 40.64))
-    (stroke (width 0) (type default) (color 0 0 0 0))
-  )
   (wire (pts (xy 186.055 31.75) (xy 180.975 31.75))
     (stroke (width 0) (type default) (color 0 0 0 0))
@@
   )
   (wire (pts (xy 106.68 127) (xy 113.665 127))
-    (stroke (width 0) (type default) (color 0 0 0 0))
-  )
-  (wire (pts (xy 170.815 45.72) (xy 170.815 43.18))
     (stroke (width 0) (type default) (color 0 0 0 0))
   )
@@
     (pin "2")
   )
-  (symbol (lib_id "Connector:USB_C_Receptacle_USB2.0") (at 155.575 40.64 0) (unit 1)
+  (symbol (lib_id "RevK:USB-C") (at 155.575 40.64 0) (unit 1)
     (in_bom yes) (on_board yes)
     (property "Reference" "J3" (id 0) (at 158.2928 18.6182 0))
     (property "Value" "USB-C" (id 1) (at 158.2928 20.9296 0))
-    (property "Footprint" "RevK:USC16-TR-Round" (id 2) (at 159.385 40.64 0)
-      (effects (font (size 1.27 1.27)) hide)
-    )
-    (property "Datasheet" "https://www.usb.org/sites/default/files/documents/usb_type-c.zip" (id 3) (at 159.385 40.64 0)
+    (property "Footprint" "RevK:USC16-TR-Round" (id 2) (at 155.575 20.32 0)
+      (effects (font (size 1.27 1.27)) hide)
+    )
+    (property "Datasheet" "https://www.usb.org/sites/default/files/documents/usb_type-c.zip" (id 3) (at 155.575 17.78 0)
       (effects (font (size 1.27 1.27)) hide)
     )
@@
     (pin "2")
   )
-  (symbol (lib_id "Connector_Generic:Conn_01x02") (at 55.88 138.43 0) (mirror y) (unit 1)
+  (symbol (lib_id "RevK:PowerIn") (at 55.88 138.43 0) (mirror y) (unit 1)
     (in_bom yes) (on_board yes)
     (property "Reference" "J1" (id 0) (at 55.88 135.89 0))
-    (property "Value" "DC" (id 1) (at 53.34 139.7 90))
-    (property "Footprint" "RevK:Molex_MiniSPOX_H2RA" (id 2) (at 55.88 138.43 0)
-      (effects (font (size 1.27 1.27)) hide)
-    )
+    (property "Value" "DC" (id 1) (at 48.26 139.7 90))
+    (property "Footprint" "RevK:Molex_MiniSPOX_H2RA" (id 2) (at 55.88 133.35 0)
+      (effects (font (size 1.27 1.27)) hide)
+    )

Commit message: Clean up
Parts:
- JP1, JP2: now left out of the parts list
Changed lines of the file:
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@@
   )
   (symbol (lib_id "Jumper:Jumper_2_Open") (at 59.055 130.175 0) (unit 1)
-    (in_bom yes) (on_board yes) (fields_autoplaced)
+    (in_bom no) (on_board yes) (fields_autoplaced)
     (property "Reference" "JP2" (id 0) (at 59.055 124.8242 0))
     (property "Value" "Jumper_2_Open" (id 1) (at 59.055 127.3611 0))
@@
   )
   (symbol (lib_id "Jumper:Jumper_2_Open") (at 59.055 122.555 0) (unit 1)
-    (in_bom yes) (on_board yes) (fields_autoplaced)
+    (in_bom no) (on_board yes) (fields_autoplaced)
     (property "Reference" "JP1" (id 0) (at 59.055 117.2042 0))
     (property "Value" "Jumper_2_Open" (id 1) (at 59.055 119.7411 0))
