File: KiCad/Generic01.kicad_pcb (KiCad board)
At the start: 2 copper layers, 13.2 x 18 mm, 3 parts, among them J1 Header, U1 ESP32-PICO-MINI-02

Commit message: Footprint update
Routing:
- net GND: track 3.90 -> 0.00 mm
Changed lines of the file:
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@@
       (effects (font (size 1 1) (thickness 0.15)))
+    )
+    (fp_text user "From PCB" (at 11 -8.2 270 unlocked) (layer "F.Fab")
+      (effects (font (size 0.5 0.5) (thickness 0.1)))
+    )
+    (fp_text user "Min 5mm" (at 10.2 -8.2 270 unlocked) (layer "F.Fab")
+      (effects (font (size 0.5 0.5) (thickness 0.1)))
+    )
+    (fp_text user "Max 2mm" (at -8.1 -8.4 270 unlocked) (layer "F.Fab")
+      (effects (font (size 0.5 0.5) (thickness 0.1)))
+    )
+    (fp_text user "Max 1mm" (at 0 -11.5 180 unlocked) (layer "F.Fab")
+      (effects (font (size 0.5 0.5) (thickness 0.1)))
     )
     (fp_text user "ANTENNA" (at -3 -7.7) (layer "F.Fab")
@@
       (effects (font (size 0.5 0.5) (thickness 0.1)))
     )
-    (fp_text user "Min 5mm" (at 10.2 -8.2 270 unlocked) (layer "F.Fab")
-      (effects (font (size 0.5 0.5) (thickness 0.1)))
-    )
-    (fp_text user "Max 2mm" (at -8.1 -8.4 270 unlocked) (layer "F.Fab")
-      (effects (font (size 0.5 0.5) (thickness 0.1)))
-    )
-    (fp_text user "Max 1mm" (at 0 -11.5 180 unlocked) (layer "F.Fab")
-      (effects (font (size 0.5 0.5) (thickness 0.1)))
-    )
-    (fp_text user "From PCB" (at 11 -8.2 270 unlocked) (layer "F.Fab")
-      (effects (font (size 0.5 0.5) (thickness 0.1)))
-    )
-    (fp_poly (pts
-        (xy -1.225 -1.225)
-        (xy -1.225 -2.675)
-        (xy -2.075 -2.675)
-        (xy -2.675 -2.075)
-        (xy -2.675 -1.225)
-      ) (layer "F.Paste") (width 0.01) (fill solid))
-    (fp_poly (pts
-        (xy -1.125 -1.125)
-        (xy -1.125 -2.775)
-        (xy -2.175 -2.775)
-        (xy -2.775 -2.175)
-        (xy -2.775 -1.125)
-      ) (layer "F.Mask") (width 0.01) (fill solid))
+    (fp_line (start -6.6 5.6) (end 6.6 5.6) (layer "F.CrtYd") (width 0.05))
+    (fp_line (start 6.6 5.6) (end 6.6 -11) (layer "F.CrtYd") (width 0.05))
+    (fp_line (start 6.6 -11) (end -6.6 -11) (layer "F.CrtYd") (width 0.05))
     (fp_line (start -6.6 -11) (end -6.6 5.6) (layer "F.CrtYd") (width 0.05))
-    (fp_line (start 6.6 5.6) (end 6.6 -11) (layer "F.CrtYd") (width 0.05))
-    (fp_line (start -6.6 5.6) (end 6.6 5.6) (layer "F.CrtYd") (width 0.05))
-    (fp_line (start 6.6 -11) (end -6.6 -11) (layer "F.CrtYd") (width 0.05))
+    (fp_line (start -6.6 -5.6) (end 6.6 -5.6) (layer "F.Fab") (width 0.127))
+    (fp_line (start 11.6 -12) (end -8.6 -12) (layer "F.Fab") (width 0.1))
     (fp_line (start 6.6 -11) (end 11.6 -11) (layer "F.Fab") (width 0.1))
     (fp_line (start -6.6 -5.6) (end -6.6 -11) (layer "F.Fab") (width 0.127))
+    (fp_line (start -8.6 -11) (end -8.6 -5.6) (layer "F.Fab") (width 0.1))
+    (fp_line (start 6.6 -11) (end 6.6 -5.6) (layer "F.Fab") (width 0.127))
+    (fp_line (start 6.6 5.6) (end -6.6 5.6) (layer "F.Fab") (width 0.127))
+    (fp_line (start 11.6 -12) (end 15.1 -12) (layer "F.Fab") (width 0.1))
+    (fp_line (start 11.6 -11) (end 11.6 -5.6) (layer "F.Fab") (width 0.1))
     (fp_line (start -6.6 -11) (end -8.6 -11) (layer "F.Fab") (width 0.1))
+    (fp_line (start -6.6 -11) (end 6.6 -11) (layer "F.Fab") (width 0.127))
+    (fp_line (start -8.6 -5.6) (end -6.6 -5.6) (layer "F.Fab") (width 0.1))
+    (fp_line (start 6.6 -5.6) (end 6.6 5.6) (layer "F.Fab") (width 0.127))
+    (fp_line (start -8.6 -12) (end -8.6 -11) (layer "F.Fab") (width 0.1))
     (fp_line (start -8.6 -5.6) (end -8.6 -2.3) (layer "F.Fab") (width 0.1))
-    (fp_line (start 6.6 5.6) (end -6.6 5.6) (layer "F.Fab") (width 0.127))
-    (fp_line (start -8.6 -11) (end -8.6 -5.6) (layer "F.Fab") (width 0.1))
-    (fp_line (start 11.6 -11) (end 11.6 -5.6) (layer "F.Fab") (width 0.1))
+    (fp_line (start 11.6 -11) (end 11.6 -12) (layer "F.Fab") (width 0.1))
     (fp_line (start 11.6 -5.6) (end 6.6 -5.6) (layer "F.Fab") (width 0.1))
-    (fp_line (start -8.6 -12) (end -8.6 -11) (layer "F.Fab") (width 0.1))
-    (fp_line (start 6.6 -11) (end 6.6 -5.6) (layer "F.Fab") (width 0.127))
-    (fp_line (start -8.6 -5.6) (end -6.6 -5.6) (layer "F.Fab") (width 0.1))
-    (fp_line (start -6.6 -11) (end 6.6 -11) (layer "F.Fab") (width 0.127))
-    (fp_line (start 6.6 -5.6) (end 6.6 5.6) (layer "F.Fab") (width 0.127))
     (fp_line (start -6.6 5.6) (end -6.6 -5.6) (layer "F.Fab") (width 0.127))
-    (fp_line (start 11.6 -12) (end -8.6 -12) (layer "F.Fab") (width 0.1))
-    (fp_line (start 11.6 -12) (end 15.1 -12) (layer "F.Fab") (width 0.1))
-    (fp_line (start -6.6 -5.6) (end 6.6 -5.6) (layer "F.Fab") (width 0.127))
-    (fp_line (start 11.6 -11) (end 11.6 -12) (layer "F.Fab") (width 0.1))
     (pad "1" smd rect (at -5.9 -4 180) (size 0.8 0.4) (layers "F.Cu" "F.Paste" "F.Mask")
       (net 2 "GND") (pinfunction "GND") (pintype "power_in"))
@@
     (pad "48" smd rect (at -4.8 -4.9 180) (size 0.4 0.8) (layers "F.Cu" "F.Paste" "F.Mask")
       (net 2 "GND") (pinfunction "GND") (pintype "power_in"))
+    (pad "49" smd rect (at 0 1.975 180) (size 1.45 1.45) (layers "F.Cu" "F.Paste" "F.Mask")
+      (net 2 "GND") (pinfunction "GND") (pintype "power_in"))
+    (pad "49" smd rect (at 1.975 -1.975 180) (size 1.45 1.45) (layers "F.Cu" "F.Paste" "F.Mask")
+      (net 2 "GND") (pinfunction "GND") (pintype "power_in"))
+    (pad "49" smd roundrect (at -1.975 -1.975 180) (size 1.45 1.45) (layers "F.Cu" "F.Paste" "F.Mask") (roundrect_rratio 0)
+      (chamfer_ratio 0.41) (chamfer top_left)
+      (net 2 "GND") (pinfunction "GND") (pintype "power_in"))
     (pad "49" smd rect (at 0 0 180) (size 1.45 1.45) (layers "F.Cu" "F.Paste" "F.Mask")
       (net 2 "GND") (pinfunction "GND") (pintype "power_in"))
+    (pad "49" smd rect (at 1.975 1.975 180) (size 1.45 1.45) (layers "F.Cu" "F.Paste" "F.Mask")
+      (net 2 "GND") (pinfunction "GND") (pintype "power_in"))
+    (pad "49" smd rect (at -1.975 1.975 180) (size 1.45 1.45) (layers "F.Cu" "F.Paste" "F.Mask")
+      (net 2 "GND") (pinfunction "GND") (pintype "power_in"))
+    (pad "49" smd rect (at 0 -1.975 180) (size 1.45 1.45) (layers "F.Cu" "F.Paste" "F.Mask")
+      (net 2 "GND") (pinfunction "GND") (pintype "power_in"))
+    (pad "49" smd rect (at -1.975 0 180) (size 1.45 1.45) (layers "F.Cu" "F.Paste" "F.Mask")
+      (net 2 "GND") (pinfunction "GND") (pintype "power_in"))
+    (pad "49" smd rect (at 1.975 0 180) (size 1.45 1.45) (layers "F.Cu" "F.Paste" "F.Mask")
+      (net 2 "GND") (pinfunction "GND") (pintype "power_in"))
     (pad "50" smd rect (at 5.95 -4.95 180) (size 0.7 0.7) (layers "F.Cu" "F.Paste" "F.Mask")
       (net 2 "GND") (pinfunction "GND") (pintype "power_in"))
@@
     (pad "53" smd rect (at -5.95 -4.95 180) (size 0.7 0.7) (layers "F.Cu" "F.Paste" "F.Mask")
       (net 2 "GND") (pinfunction "GND") (pintype "power_in"))
-    (pad "54" smd rect (at -1.95 0 180) (size 1.45 1.45) (layers "F.Cu" "F.Paste" "F.Mask")
-      (net 2 "GND") (pinfunction "GND") (pintype "power_in"))
-    (pad "55" smd rect (at -1.95 1.95 180) (size 1.45 1.45) (layers "F.Cu" "F.Paste" "F.Mask")
-      (net 2 "GND") (pinfunction "GND") (pintype "power_in"))
-    (pad "56" smd rect (at 0 1.95 180) (size 1.45 1.45) (layers "F.Cu" "F.Paste" "F.Mask")
-      (net 2 "GND") (pinfunction "GND") (pintype "power_in"))
-    (pad "57" smd rect (at 1.95 1.95 180) (size 1.45 1.45) (layers "F.Cu" "F.Paste" "F.Mask")
-      (net 2 "GND") (pinfunction "GND") (pintype "power_in"))
-    (pad "58" smd rect (at 1.95 0 180) (size 1.45 1.45) (layers "F.Cu" "F.Paste" "F.Mask")
-      (net 2 "GND") (pinfunction "GND") (pintype "power_in"))
-    (pad "59" smd rect (at 1.95 -1.95 180) (size 1.45 1.45) (layers "F.Cu" "F.Paste" "F.Mask")
-      (net 2 "GND") (pinfunction "GND") (pintype "power_in"))
-    (pad "60" smd rect (at 0 -1.95 180) (size 1.45 1.45) (layers "F.Cu" "F.Paste" "F.Mask")
-      (net 2 "GND") (pinfunction "GND") (pintype "power_in"))
-    (pad "61" smd custom (at -1.95 -1.95 180) (size 0.5 0.5) (layers "F.Cu")
-      (net 2 "GND") (pinfunction "GND") (pintype "power_in") (zone_connect 0)
-      (options (clearance outline) (anchor rect))
-      (primitives
-        (gr_poly (pts
-            (xy 0.725 0.725)
-            (xy 0.725 -0.725)
-            (xy -0.125 -0.725)
-            (xy -0.725 -0.125)
-            (xy -0.725 0.725)
-          ) (width 0.01) (fill yes))
-      ))
-    (zone (net 0) (net_name "") (layer "F.Cu") (hatch full 0.508)
+    (zone (net 0) (net_name "") (layers *.Cu) (hatch full 0.508)
       (connect_pads (clearance 0))
       (min_thickness 0.01)
-      (keepout (tracks not_allowed) (vias not_allowed) (pads not_allowed ) (copperpour not_allowed) (footprints allowed))
+      (keepout (tracks allowed) (vias not_allowed) (pads allowed ) (copperpour allowed) (footprints allowed))
       (fill (thermal_gap 0.508) (thermal_bridge_width 0.508))
       (polygon
@@
       )
     )
-    (zone (net 0) (net_name "") (layers *.Cu) (hatch full 0.508)
+    (zone (net 0) (net_name "") (layer "F.Cu") (hatch full 0.508)
       (connect_pads (clearance 0))
       (min_thickness 0.01)
-      (keepout (tracks allowed) (vias not_allowed) (pads allowed ) (copperpour allowed) (footprints allowed))
+      (keepout (tracks not_allowed) (vias not_allowed) (pads not_allowed ) (copperpour not_allowed) (footprints allowed))
       (fill (thermal_gap 0.508) (thermal_bridge_width 0.508))
       (polygon
@@
   (arc (start 149.41 105.06) (mid 149.065994 105.890505) (end 148.235489 106.234511) (width 0.25) (layer "B.Cu") (net 1))
   (arc (start 144 109) (mid 142.40901 109.65901) (end 141.75 111.25) (width 0.25) (layer "B.Cu") (net 1))
-  (segment (start 147.55 115.4) (end 147.55 117.35) (width 0.25) (layer "F.Cu") (net 2))
-  (segment (start 145.6 117.35) (end 147.55 117.35) (width 0.25) (layer "F.Cu") (net 2))
   (segment (start 143.825489 108.774511) (end 145.695489 108.774511) (width 0.25) (layer "F.Cu") (net 3))
   (segment (start 142.4 110.2) (end 143.825489 108.774511) (width 0.25) (layer "F.Cu") (net 3))

Commit message: Tidy
Other:
- board text added: "www.me.uk"
Changed lines of the file:
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@@
       (effects (font (size 1 1) (thickness 0.15)))
     )
-    (fp_text user "From PCB" (at 11 -8.2 270 unlocked) (layer "F.Fab")
-      (effects (font (size 0.5 0.5) (thickness 0.1)))
-    )
-    (fp_text user "Min 5mm" (at 10.2 -8.2 270 unlocked) (layer "F.Fab")
-      (effects (font (size 0.5 0.5) (thickness 0.1)))
-    )
-    (fp_text user "Max 2mm" (at -8.1 -8.4 270 unlocked) (layer "F.Fab")
-      (effects (font (size 0.5 0.5) (thickness 0.1)))
-    )
-    (fp_text user "Max 1mm" (at 0 -11.5 180 unlocked) (layer "F.Fab")
-      (effects (font (size 0.5 0.5) (thickness 0.1)))
+    (fp_text user "${DATE}" (at 0 -3.6 180 unlocked) (layer "F.SilkS")
+      (effects (font (size 0.75 0.75) (thickness 0.1)))
     )
     (fp_text user "ANTENNA" (at -3 -7.7) (layer "F.Fab")
@@
       (effects (font (size 0.5 0.5) (thickness 0.1)))
     )
+    (fp_text user "Max 2mm" (at -8.1 -8.4 270 unlocked) (layer "F.Fab")
+      (effects (font (size 0.5 0.5) (thickness 0.1)))
+    )
+    (fp_text user "Max 1mm" (at 0 -11.5 180 unlocked) (layer "F.Fab")
+      (effects (font (size 0.5 0.5) (thickness 0.1)))
+    )
+    (fp_text user "Min 5mm" (at 10.2 -8.2 270 unlocked) (layer "F.Fab")
+      (effects (font (size 0.5 0.5) (thickness 0.1)))
+    )
+    (fp_text user "From PCB" (at 11 -8.2 270 unlocked) (layer "F.Fab")
+      (effects (font (size 0.5 0.5) (thickness 0.1)))
+    )
+    (fp_line (start 6.6 -11) (end -6.6 -11) (layer "F.CrtYd") (width 0.05))
+    (fp_line (start -6.6 -11) (end -6.6 5.6) (layer "F.CrtYd") (width 0.05))
     (fp_line (start -6.6 5.6) (end 6.6 5.6) (layer "F.CrtYd") (width 0.05))
     (fp_line (start 6.6 5.6) (end 6.6 -11) (layer "F.CrtYd") (width 0.05))
-    (fp_line (start 6.6 -11) (end -6.6 -11) (layer "F.CrtYd") (width 0.05))
-    (fp_line (start -6.6 -11) (end -6.6 5.6) (layer "F.CrtYd") (width 0.05))
-    (fp_line (start -6.6 -5.6) (end 6.6 -5.6) (layer "F.Fab") (width 0.127))
+    (fp_line (start -6.6 -11) (end -8.6 -11) (layer "F.Fab") (width 0.1))
+    (fp_line (start 11.6 -5.6) (end 6.6 -5.6) (layer "F.Fab") (width 0.1))
     (fp_line (start 11.6 -12) (end -8.6 -12) (layer "F.Fab") (width 0.1))
+    (fp_line (start -8.6 -11) (end -8.6 -5.6) (layer "F.Fab") (width 0.1))
+    (fp_line (start 11.6 -11) (end 11.6 -12) (layer "F.Fab") (width 0.1))
+    (fp_line (start -6.6 -5.6) (end -6.6 -11) (layer "F.Fab") (width 0.127))
     (fp_line (start 6.6 -11) (end 11.6 -11) (layer "F.Fab") (width 0.1))
-    (fp_line (start -6.6 -5.6) (end -6.6 -11) (layer "F.Fab") (width 0.127))
-    (fp_line (start -8.6 -11) (end -8.6 -5.6) (layer "F.Fab") (width 0.1))
-    (fp_line (start 6.6 -11) (end 6.6 -5.6) (layer "F.Fab") (width 0.127))
-    (fp_line (start 6.6 5.6) (end -6.6 5.6) (layer "F.Fab") (width 0.127))
-    (fp_line (start 11.6 -12) (end 15.1 -12) (layer "F.Fab") (width 0.1))
-    (fp_line (start 11.6 -11) (end 11.6 -5.6) (layer "F.Fab") (width 0.1))
-    (fp_line (start -6.6 -11) (end -8.6 -11) (layer "F.Fab") (width 0.1))
-    (fp_line (start -6.6 -11) (end 6.6 -11) (layer "F.Fab") (width 0.127))
     (fp_line (start -8.6 -5.6) (end -6.6 -5.6) (layer "F.Fab") (width 0.1))
     (fp_line (start 6.6 -5.6) (end 6.6 5.6) (layer "F.Fab") (width 0.127))
+    (fp_line (start 6.6 5.6) (end -6.6 5.6) (layer "F.Fab") (width 0.127))
+    (fp_line (start 6.6 -11) (end 6.6 -5.6) (layer "F.Fab") (width 0.127))
+    (fp_line (start -6.6 5.6) (end -6.6 -5.6) (layer "F.Fab") (width 0.127))
+    (fp_line (start -8.6 -5.6) (end -8.6 -2.3) (layer "F.Fab") (width 0.1))
+    (fp_line (start -6.6 -11) (end 6.6 -11) (layer "F.Fab") (width 0.127))
+    (fp_line (start 11.6 -11) (end 11.6 -5.6) (layer "F.Fab") (width 0.1))
     (fp_line (start -8.6 -12) (end -8.6 -11) (layer "F.Fab") (width 0.1))
-    (fp_line (start -8.6 -5.6) (end -8.6 -2.3) (layer "F.Fab") (width 0.1))
-    (fp_line (start 11.6 -11) (end 11.6 -12) (layer "F.Fab") (width 0.1))
-    (fp_line (start 11.6 -5.6) (end 6.6 -5.6) (layer "F.Fab") (width 0.1))
-    (fp_line (start -6.6 5.6) (end -6.6 -5.6) (layer "F.Fab") (width 0.127))
+    (fp_line (start 11.6 -12) (end 15.1 -12) (layer "F.Fab") (width 0.1))
+    (fp_line (start -6.6 -5.6) (end 6.6 -5.6) (layer "F.Fab") (width 0.127))
     (pad "1" smd rect (at -5.9 -4 180) (size 0.8 0.4) (layers "F.Cu" "F.Paste" "F.Mask")
       (net 2 "GND") (pinfunction "GND") (pintype "power_in"))
@@
     (pad "48" smd rect (at -4.8 -4.9 180) (size 0.4 0.8) (layers "F.Cu" "F.Paste" "F.Mask")
       (net 2 "GND") (pinfunction "GND") (pintype "power_in"))
+    (pad "49" smd rect (at -1.975 0 180) (size 1.45 1.45) (layers "F.Cu" "F.Paste" "F.Mask")
+      (net 2 "GND") (pinfunction "GND") (pintype "power_in"))
+    (pad "49" smd rect (at 0 0 180) (size 1.45 1.45) (layers "F.Cu" "F.Paste" "F.Mask")
+      (net 2 "GND") (pinfunction "GND") (pintype "power_in"))
+    (pad "49" smd rect (at 1.975 -1.975 180) (size 1.45 1.45) (layers "F.Cu" "F.Paste" "F.Mask")
+      (net 2 "GND") (pinfunction "GND") (pintype "power_in"))
     (pad "49" smd rect (at 0 1.975 180) (size 1.45 1.45) (layers "F.Cu" "F.Paste" "F.Mask")
-      (net 2 "GND") (pinfunction "GND") (pintype "power_in"))
-    (pad "49" smd rect (at 1.975 -1.975 180) (size 1.45 1.45) (layers "F.Cu" "F.Paste" "F.Mask")
       (net 2 "GND") (pinfunction "GND") (pintype "power_in"))
     (pad "49" smd roundrect (at -1.975 -1.975 180) (size 1.45 1.45) (layers "F.Cu" "F.Paste" "F.Mask") (roundrect_rratio 0)
       (chamfer_ratio 0.41) (chamfer top_left)
       (net 2 "GND") (pinfunction "GND") (pintype "power_in"))
-    (pad "49" smd rect (at 0 0 180) (size 1.45 1.45) (layers "F.Cu" "F.Paste" "F.Mask")
+    (pad "49" smd rect (at 1.975 0 180) (size 1.45 1.45) (layers "F.Cu" "F.Paste" "F.Mask")
+      (net 2 "GND") (pinfunction "GND") (pintype "power_in"))
+    (pad "49" smd rect (at -1.975 1.975 180) (size 1.45 1.45) (layers "F.Cu" "F.Paste" "F.Mask")
       (net 2 "GND") (pinfunction "GND") (pintype "power_in"))
     (pad "49" smd rect (at 1.975 1.975 180) (size 1.45 1.45) (layers "F.Cu" "F.Paste" "F.Mask")
       (net 2 "GND") (pinfunction "GND") (pintype "power_in"))
-    (pad "49" smd rect (at -1.975 1.975 180) (size 1.45 1.45) (layers "F.Cu" "F.Paste" "F.Mask")
-      (net 2 "GND") (pinfunction "GND") (pintype "power_in"))
     (pad "49" smd rect (at 0 -1.975 180) (size 1.45 1.45) (layers "F.Cu" "F.Paste" "F.Mask")
       (net 2 "GND") (pinfunction "GND") (pintype "power_in"))
-    (pad "49" smd rect (at -1.975 0 180) (size 1.45 1.45) (layers "F.Cu" "F.Paste" "F.Mask")
-      (net 2 "GND") (pinfunction "GND") (pintype "power_in"))
-    (pad "49" smd rect (at 1.975 0 180) (size 1.45 1.45) (layers "F.Cu" "F.Paste" "F.Mask")
-      (net 2 "GND") (pinfunction "GND") (pintype "power_in"))
     (pad "50" smd rect (at 5.95 -4.95 180) (size 0.7 0.7) (layers "F.Cu" "F.Paste" "F.Mask")
       (net 2 "GND") (pinfunction "GND") (pintype "power_in"))
@@
     (pad "53" smd rect (at -5.95 -4.95 180) (size 0.7 0.7) (layers "F.Cu" "F.Paste" "F.Mask")
       (net 2 "GND") (pinfunction "GND") (pintype "power_in"))
-    (zone (net 0) (net_name "") (layers *.Cu) (hatch full 0.508)
+    (zone (net 0) (net_name "") (layer "F.Cu") (hatch full 0.508)
       (connect_pads (clearance 0))
       (min_thickness 0.01)
-      (keepout (tracks allowed) (vias not_allowed) (pads allowed ) (copperpour allowed) (footprints allowed))
+      (keepout (tracks not_allowed) (vias not_allowed) (pads not_allowed ) (copperpour not_allowed) (footprints allowed))
       (fill (thermal_gap 0.508) (thermal_bridge_width 0.508))
       (polygon
@@
       )
     )
-    (zone (net 0) (net_name "") (layer "F.Cu") (hatch full 0.508)
+    (zone (net 0) (net_name "") (layers *.Cu) (hatch full 0.508)
       (connect_pads (clearance 0))
       (min_thickness 0.01)
-      (keepout (tracks not_allowed) (vias not_allowed) (pads not_allowed ) (copperpour not_allowed) (footprints allowed))
+      (keepout (tracks allowed) (vias not_allowed) (pads allowed ) (copperpour allowed) (footprints allowed))
       (fill (thermal_gap 0.508) (thermal_bridge_width 0.508))
       (polygon
@@
   (gr_line (start 139 103) (end 139 121) (layer "Edge.Cuts") (width 0.1))
   (gr_line (start 139 121) (end 152.2 121) (layer "Edge.Cuts") (width 0.1))
+  (gr_text "www.me.uk" (at 146.4 116.7) (layer "B.SilkS")
+    (effects (font (size 0.75 0.75) (thickness 0.1)) (justify mirror))
+  )
   (dimension (type aligned) (layer "Dwgs.User")
     (pts (xy 139 121) (xy 152.2 121))

Commit message: Tidy
Parts:
- moved Logo1 0.38 mm to (145.9, 112.8)
Other:
- board text removed: "www.me.uk"
Changed lines of the file:
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@@
   )
   (footprint "RevK:AJK" (layer "B.Cu")
-    (at 145.9 113.125 180)
+    (at 145.9 112.75 180)
     (property "Note" "Non part, PCB printed")
     (property "Sheetfile" "Generic01.kicad_sch")
@@
       (effects (font (size 1 1) (thickness 0.15)) (justify mirror))
     )
+    (fp_text user "www.me.uk" (at -0.58 -3.75 unlocked) (layer "B.SilkS")
+      (effects (font (size 0.65 0.65) (thickness 0.1)) (justify mirror))
+    )
+    (fp_line (start -0.85 -1.95) (end -0.75 -1.95) (layer "B.Cu") (width 0.08))
+    (fp_line (start 0 0) (end 1.8 -2.1) (layer "B.Cu") (width 0.25))
+    (fp_line (start -0.85 -1.95) (end -0.85 -2.25) (layer "B.Cu") (width 0.08))
+    (fp_line (start -0.85 -2.11) (end -0.75 -2.11) (layer "B.Cu") (width 0.08))
+    (fp_line (start -0.75 -2.11) (end -0.65 -2.25) (layer "B.Cu") (width 0.08))
     (fp_line (start 1.8 2) (end 0 0) (layer "B.Cu") (width 0.25))
-    (fp_line (start -0.85 -1.95) (end -0.75 -1.95) (layer "B.Cu") (width 0.08))
-    (fp_line (start -0.85 -2.11) (end -0.75 -2.11) (layer "B.Cu") (width 0.08))
     (fp_line (start 0 2.1) (end 0 -2.1) (layer "B.Cu") (width 0.25))
-    (fp_line (start -0.75 -2.11) (end -0.65 -2.25) (layer "B.Cu") (width 0.08))
     (fp_line (start 0 2.1) (end -3 -2.1) (layer "B.Cu") (width 0.25))
     (fp_line (start 0 0) (end -1.5 0) (layer "B.Cu") (width 0.25))
-    (fp_line (start -0.85 -1.95) (end -0.85 -2.25) (layer "B.Cu") (width 0.08))
-    (fp_line (start 0 0) (end 1.8 -2.1) (layer "B.Cu") (width 0.25))
+    (fp_arc (start -0.75 -2.11) (mid -0.67 -2.03) (end -0.75 -1.95) (layer "B.Cu") (width 0.08))
     (fp_arc (start -1.5 -2.1) (mid -0.75 -2.85) (end 0 -2.1) (layer "B.Cu") (width 0.25))
-    (fp_arc (start -0.75 -2.11) (mid -0.67 -2.03) (end -0.75 -1.95) (layer "B.Cu") (width 0.08))
     (fp_circle (center -0.77 -2.11) (end -0.47 -2.11) (layer "B.Cu") (width 0.08) (fill none))
+    (fp_line (start 0 2.1) (end -3 -2.1) (layer "B.Mask") (width 0.45))
+    (fp_line (start 0 2.1) (end 0 -2.1) (layer "B.Mask") (width 0.45))
     (fp_line (start 0 0) (end 1.8 -2.1) (layer "B.Mask") (width 0.45))
     (fp_line (start 1.8 2) (end 0 0) (layer "B.Mask") (width 0.45))
-    (fp_line (start 0 2.1) (end 0 -2.1) (layer "B.Mask") (width 0.45))
     (fp_line (start 0 0) (end -1.5 0) (layer "B.Mask") (width 0.45))
-    (fp_line (start 0 2.1) (end -3 -2.1) (layer "B.Mask") (width 0.45))
     (fp_arc (start -1.5 -2.1) (mid -0.75 -2.85) (end 0 -2.1) (layer "B.Mask") (width 0.45))
   )
@@
   (gr_line (start 139 103) (end 139 121) (layer "Edge.Cuts") (width 0.1))
   (gr_line (start 139 121) (end 152.2 121) (layer "Edge.Cuts") (width 0.1))
-  (gr_text "www.me.uk" (at 146.4 116.7) (layer "B.SilkS")
-    (effects (font (size 0.75 0.75) (thickness 0.1)) (justify mirror))
-  )
   (dimension (type aligned) (layer "Dwgs.User")
     (pts (xy 139 121) (xy 152.2 121))
