File: KiCad/Generic4.kicad_pcb (KiCad board)
At the start: 2 copper layers, 13.2 x 19.5 mm, 11 parts, among them J1 I/O, J2 SPOX, U1 ESP32-PICO-MINI-02, U2 LMR16006+FB

Commit message: Tidy
Parts:
- added D1: RGB, RevK:LED-RGB-1.6x1.6, B.Cu at (105.2, 42.7)
- added R1: 680R, RevK:R_0603, B.Cu at (104.8, 46.8)
- added R2: 2K, RevK:R_0603, B.Cu at (104.8, 44.8)
- added R3: 220R, RevK:R_0603, B.Cu at (104.8, 49.0)
- moved R5 3.72 mm to (102.2, 39.5), turned to 0 degrees
- moved U2 1.21 mm to (100.2, 42.2)
- moved R4 0.76 mm to (105.0, 39.5), turned to 180 degrees
- renumbered D1 to D2, R1 to R4, R2 to R5
Connections:
- U1 pad 26: unconnected-(U1-Pad26) -> B
- U1 pad 33: unconnected-(U1-Pad33) -> R
- U1 pad 34: unconnected-(U1-Pad34) -> G
Routing:
- net GND: track 67.1 -> 38.7 mm, vias 1 -> 4
- net Net-(D1-Pad4): track 0.00 -> 7.60 mm
- net R: track 0.00 -> 7.00 mm, vias 0 -> 1
- net G: track 0.00 -> 6.91 mm, vias 0 -> 1
- net GPIO0: track 16.2 -> 21.9 mm, vias 0 -> 1
- net IO2: track 6.02 -> 10.8 mm
- net IO4: track 5.56 -> 9.18 mm
- net Net-(D1-Pad2): track 0.00 -> 3.54 mm
- net B: track 0.00 -> 2.59 mm, vias 0 -> 1
- net EN: track 18.0 -> 20.1 mm, vias 1 -> 2
- net IO5: track 11.8 -> 10.1 mm, vias 1 -> 0
- net Net-(D1-Pad3): track 0.00 -> 1.23 mm
- net TX: track 11.4 -> 10.2 mm
- net DC: track 12.5 -> 11.5 mm
- net IO7: track 9.13 -> 8.42 mm
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Other:
- board text removed: "${DATE}"

Commit message: Tweak
Routing:
- net B: track 2.59 -> 3.86 mm
- net IO3: track 10.4 -> 11.6 mm
- net GPIO0: track 21.9 -> 22.5 mm

Commit message: Started on Generic5
Parts:
- J1: footprint Connector_PinHeader_2.54mm:PinHeader_2x04_P2.54mm_Vertical -> Connector_PinHeader_2.54mm:PinHeader_2x05_P2.54mm_Vertical
- moved R3 4.44 mm to (105.9, 44.7), turned to -90 degrees
- moved R1 2.90 mm to (102.7, 44.7), turned to -90 degrees
- moved J1 1.27 mm to (94.9, 54.0)
- moved D1 1.14 mm to (104.9, 41.6), turned to 0 degrees
- moved U2 0.85 mm to (99.7, 41.6)
- moved R2 0.45 mm to (104.3, 44.7), turned to -90 degrees
- moved R5 0.15 mm to (102.4, 39.5)
Connections:
- J1 pad 1: GPIO0 -> GND
- J1 pad 3: IO2 -> GPIO0
- J1 pad 4: IO3 -> IO2
- J1 pad 5: IO4 -> EN
- J1 pad 6: IO5 -> IO3
- J1 pad 7: IO6 -> RX
- J1 pad 8: IO7 -> IO4
- J2 pad 3: TX -> IO6
- J2 pad 4: RX -> IO7
- U1 pad 20: IO5 -> unconnected-(U1-Pad20)
- U1 pad 26: B -> IO5
- U1 pad 27: unconnected-(U1-Pad27) -> B
- U1 pad 33: R -> G
- U1 pad 34: G -> R
Routing:
- net EN: track 20.2 -> 36.8 mm, vias 2 -> 3
- net IO2: track 10.4 -> 20.6 mm, vias 0 -> 1
- net GPIO0: track 22.5 -> 12.6 mm
- net Net-(D1-Pad4): track 7.86 -> 1.84 mm
- net IO7: track 8.17 -> 2.90 mm
- net RX: track 8.57 -> 11.5 mm
- net TX: track 9.87 -> 12.6 mm
- net IO6: track 5.34 -> 2.96 mm
- net IO3: track 11.6 -> 9.44 mm, vias 2 -> 0
- net GND: track 38.5 -> 40.1 mm, vias 4 -> 3
- net G: track 6.65 -> 5.10 mm
- net IO5: track 9.72 -> 11.1 mm, vias 0 -> 1
- net B: track 3.86 -> 2.61 mm
- net IO1: track 10.5 -> 11.2 mm, vias 2 -> 0
- net Net-(D1-Pad3): track 1.23 -> 1.92 mm
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Other:
- board text added: "0"
- board text added: "14"
- board text added: "15"
- board text added: "20"
- board text added: "25"
- board text added: "26"
- board text added: "27"
- board text added: "3.3"
- board text added: "4"
- board text added: "Rx"
- board text added: "Tx"
- board text added: "⏚"
- board text removed: "GND"
- board text removed: "GPIO0"
- board text removed: "RX"
- board text removed: "TX"

Commit message: Silkscreen
Other:
- board text added: "Generic4"
Changed lines of the file:
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@@
     (effects (font (size 0.5 0.5) (thickness 0.1)) (justify mirror))
+  )
+  (gr_text "Generic4" (at 105.75 49.75 270) (layer "B.SilkS")
+    (effects (font (size 0.75 0.75) (thickness 0.1)) (justify mirror))
   )
   (gr_text "3.3" (at 99.1 53.15 45) (layer "B.SilkS")

Commit message: DRC tidy
Parts:
- moved R2 0.25 mm to (104.5, 44.7)
- moved U2 0.20 mm to (99.8, 41.6)
- moved R5 0.12 mm to (102.5, 39.5)
- moved R3 0.05 mm to (105.8, 44.7)
Routing:
- net GND: track 40.1 -> 39.2 mm, vias 3 -> 4
Other:
- rule pad_to_mask_clearance: 0 -> 0.125

Commit message: DRC
Routing:
- net IO2: track 20.5 -> 19.7 mm
- net IO5: track 11.1 -> 10.5 mm
Changed lines of the file:
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@@
     (style (thickness 0.2) (arrow_length 1.27) (text_position_mode 0) (extension_height 0.58642) (extension_offset 0.5) keep_text_aligned)
   )
+  (segment (start 94.05 55.625) (end 93.863389 55.811611) (width 0.25) (layer "F.Cu") (net 1))
+  (segment (start 95.00104 57.725) (end 104.99896 57.725) (width 0.25) (layer "F.Cu") (net 1))
+  (segment (start 94.380528 55.294472) (end 94.05 55.625) (width 0.25) (layer "F.Cu") (net 1))
   (segment (start 94.05 49.14325) (end 94.05 53.105) (width 0.25) (layer "F.Cu") (net 1))
-  (segment (start 94.507378 57.675) (end 105 57.675) (width 0.125) (layer "F.Cu") (net 1))
-  (segment (start 93.725 56.25) (end 93.725 56.892622) (width 0.125) (layer "F.Cu") (net 1))
+  (segment (start 93.775 56.025) (end 93.775 56.817158) (width 0.125) (layer "F.Cu") (net 1))
+  (segment (start 105.95 49.14325) (end 105.95 53.023224) (width 0.25) (layer "F.Cu") (net 1))
   (segment (start 96.8 49.09325) (end 96.8 48.793748) (width 0.25) (layer "F.Cu") (net 1))
-  (segment (start 94.925 53.98) (end 94.481604 54.423396) (width 0.125) (layer "F.Cu") (net 1))
-  (segment (start 106.25 56.425) (end 106.25 49.44325) (width 0.125) (layer "F.Cu") (net 1))
+  (segment (start 106.2 53.45) (end 106.2 56.877513) (width 0.125) (layer "F.Cu") (net 1))
   (via (at 97.5405 45.25) (size 0.8) (drill 0.4) (layers "F.Cu" "B.Cu") (net 1))
   (via (at 96.1 48.093748) (size 0.8) (drill 0.4) (layers "F.Cu" "B.Cu") (net 1))
   (via (at 103.75 55.25) (size 0.8) (drill 0.4) (layers "F.Cu" "B.Cu") (free) (net 1))
   (via (at 95.95 40.625) (size 0.8) (drill 0.4) (layers "F.Cu" "B.Cu") (net 1))
-  (arc (start 106.25 49.44325) (mid 106.162132 49.231118) (end 105.95 49.14325) (width 0.125) (layer "F.Cu") (net 1))
+  (arc (start 93.863389 55.811611) (mid 93.797971 55.909515) (end 93.775 56.025) (width 0.125) (layer "F.Cu") (net 1))
+  (arc (start 106.025 57.3) (mid 105.554249 57.614546) (end 104.99896 57.725) (width 0.125) (layer "F.Cu") (net 1))
+  (arc (start 105.95 53.023224) (mid 105.982487 53.186544) (end 106.075 53.325) (width 0.25) (layer "F.Cu") (net 1))
+  (arc (start 94.925 53.98) (mid 94.783496 54.691387) (end 94.380528 55.294472) (width 0.25) (layer "F.Cu") (net 1))
+  (arc (start 93.775 56.817158) (mid 93.826979 57.07847) (end 93.975 57.3) (width 0.125) (layer "F.Cu") (net 1))
   (arc (start 96.8 48.793748) (mid 96.594975 48.298773) (end 96.1 48.093748) (width 0.25) (layer "F.Cu") (net 1))
-  (arc (start 105 57.675) (mid 105.883883 57.308883) (end 106.25 56.425) (width 0.125) (layer "F.Cu") (net 1))
-  (arc (start 94.481604 54.423396) (mid 93.921635 55.261449) (end 93.725 56.25) (width 0.125) (layer "F.Cu") (net 1))
-  (arc (start 93.725 56.892622) (mid 93.954153 57.445847) (end 94.507378 57.675) (width 0.125) (layer "F.Cu") (net 1))
+  (arc (start 106.075 53.325) (mid 106.163388 53.361612) (end 106.2 53.45) (width 0.125) (layer "F.Cu") (net 1))
   (arc (start 94.05 53.105) (mid 94.306282 53.723718) (end 94.925 53.98) (width 0.25) (layer "F.Cu") (net 1))
+  (arc (start 106.2 56.877513) (mid 106.154519 57.106161) (end 106.025 57.3) (width 0.125) (layer "F.Cu") (net 1))
+  (arc (start 93.975 57.3) (mid 94.445751 57.614546) (end 95.00104 57.725) (width 0.25) (layer "F.Cu") (net 1))
   (segment (start 99.65 39.45) (end 99.65 40.25) (width 0.25) (layer "B.Cu") (net 1))
   (segment (start 101.575 39.5) (end 101.375 39.3) (width 0.25) (layer "B.Cu") (net 1))
@@
   (segment (start 98.4 48) (end 98.3 47.9) (width 0.25) (layer "F.Cu") (net 18))
   (via (at 98.3 47.9) (size 0.8) (drill 0.4) (layers "F.Cu" "B.Cu") (net 18))
-  (segment (start 93.75 57.075) (end 93.75 48.275) (width 0.125) (layer "B.Cu") (net 18))
-  (segment (start 96.26 57.725) (end 94.4 57.725) (width 0.125) (layer "B.Cu") (net 18))
-  (segment (start 95.1 46.925) (end 97.325 46.925) (width 0.125) (layer "B.Cu") (net 18))
-  (arc (start 97.325 46.925) (mid 98.014429 47.210571) (end 98.3 47.9) (width 0.125) (layer "B.Cu") (net 18))
-  (arc (start 94.4 57.725) (mid 93.940381 57.534619) (end 93.75 57.075) (width 0.125) (layer "B.Cu") (net 18))
-  (arc (start 93.75 48.275) (mid 94.145406 47.320406) (end 95.1 46.925) (width 0.125) (layer "B.Cu") (net 18))
-  (arc (start 97.465 56.52) (mid 97.112064 57.372064) (end 96.26 57.725) (width 0.125) (layer "B.Cu") (net 18))
+  (segment (start 93.85 49.2186) (end 93.85 52.805489) (width 0.25) (layer "B.Cu") (net 18))
+  (segment (start 94.693747 47.393747) (end 94.543747 47.543747) (width 0.25) (layer "B.Cu") (net 18))
+  (segment (start 97.275 46.875) (end 95.946113 46.875) (width 0.25) (layer "B.Cu") (net 18))
+  (segment (start 95.975 57.65) (end 95.65 57.65) (width 0.25) (layer "B.Cu") (net 18))
+  (segment (start 94.6 57.65) (end 95.65 57.65) (width 0.125) (layer "B.Cu") (net 18))
+  (segment (start 96.589559 57.395442) (end 97.465 56.52) (width 0.25) (layer "B.Cu") (net 18))
+  (segment (start 93.812989 52.8425) (end 93.812989 56.862989) (width 0.125) (layer "B.Cu") (net 18))
+  (segment (start 93.85 52.805489) (end 93.812989 52.8425) (width 0.125) (layer "B.Cu") (net 18))
+  (arc (start 93.812989 56.862989) (mid 94.043499 57.41949) (end 94.6 57.65) (width 0.125) (layer "B.Cu") (net 18))
+  (arc (start 95.946113 46.875) (mid 95.268338 47.009818) (end 94.693747 47.393747) (width 0.25) (layer "B.Cu") (net 18))
+  (arc (start 95.975 57.65) (mid 96.307597 57.583842) (end 96.589559 57.395442) (width 0.25) (layer "B.Cu") (net 18))
+  (arc (start 98.3 47.9) (mid 97.999784 47.175216) (end 97.275 46.875) (width 0.25) (layer "B.Cu") (net 18))
+  (arc (start 93.85 49.2186) (mid 94.030299 48.312176) (end 94.543747 47.543747) (width 0.25) (layer "B.Cu") (net 18))
   (segment (start 97.34325 50) (end 95.602507 50) (width 0.25) (layer "F.Cu") (net 20))
   (segment (start 96.290489 52.996467) (end 96.290489 55.154511) (width 0.25) (layer "F.Cu") (net 20))
@@
   (via (at 104.9 48.093748) (size 0.8) (drill 0.4) (layers "F.Cu" "B.Cu") (net 26))
   (arc (start 105.600498 47.39325) (mid 105.105171 47.598421) (end 104.9 48.093748) (width 0.25) (layer "F.Cu") (net 26))
-  (segment (start 106.2 55.405) (end 106.2 49.393748) (width 0.125) (layer "B.Cu") (net 26))
-  (arc (start 106.2 49.393748) (mid 105.819239 48.474509) (end 104.9 48.093748) (width 0.125) (layer "B.Cu") (net 26))
-  (arc (start 105.085 56.52) (mid 105.873424 56.193424) (end 106.2 55.405) (width 0.125) (layer "B.Cu") (net 26))
+  (segment (start 105.085 56.52) (end 105.464357 56.140643) (width 0.25) (layer "B.Cu") (net 26))
+  (segment (start 106.15 51.111514) (end 106.15 53.38399) (width 0.25) (layer "B.Cu") (net 26))
+  (segment (start 106.15 53.38399) (end 106.192968 53.426958) (width 0.125) (layer "B.Cu") (net 26))
+  (segment (start 106.275 54.183579) (end 106.275 53.625) (width 0.125) (layer "B.Cu") (net 26))
+  (arc (start 106.192968 53.426958) (mid 106.25368 53.51782) (end 106.275 53.625) (width 0.125) (layer "B.Cu") (net 26))
+  (arc (start 106.175 54.425) (mid 106.249011 54.314235) (end 106.275 54.183579) (width 0.125) (layer "B.Cu") (net 26))
+  (arc (start 105.464357 56.140643) (mid 105.99031 55.353499) (end 106.175 54.425) (width 0.25) (layer "B.Cu") (net 26))
+  (arc (start 104.9 48.093748) (mid 105.825135 49.478311) (end 106.15 51.111514) (width 0.25) (layer "B.Cu") (net 26))
   (segment (start 102.4 49.09325) (end 102.4 50.29) (width 0.25) (layer "F.Cu") (net 27))
   (arc (start 102.4 50.29) (mid 102.063173 51.103173) (end 101.25 51.44) (width 0.25) (layer "F.Cu") (net 27))
@@
   (arc (start 104.375127 41.624873) (mid 105.074745 41.157404) (end 105.9 40.99325) (width 0.25) (layer "F.Cu") (net 30))
   (arc (start 103.8 43.013172) (mid 103.949437 42.261899) (end 104.375 41.625) (width 0.25) (layer "F.Cu") (net 30))
-  (segment (start 103.49952 43.77452) (end 103.49952 43.35048) (width 0.25) (layer "B.Cu") (net 30))
+  (segment (start 103.49952 44.296271) (end 103.49952 43.35048) (width 0.25) (layer "B.Cu") (net 30))
   (segment (start 103.49952 44.296271) (end 102.7 45.095791) (width 0.25) (layer "B.Cu") (net 30))
   (segment (start 102.7 45.095791) (end 102.7 45.525) (width 0.25) (layer "B.Cu") (net 30))
-  (segment (start 103.49952 43.77452) (end 103.49952 44.296271) (width 0.25) (layer "B.Cu") (net 30))
   (arc (start 103.49952 43.35048) (mid 103.587529 43.138009) (end 103.8 43.05) (width 0.25) (layer "B.Cu") (net 30))
   (segment (start 105.600355 41.79325) (end 105.9 41.79325) (width 0.25) (layer "F.Cu") (net 31))

Commit message: DRC tweak
Routing:
- net GND: track 39.2 -> 43.8 mm
Other:
- rule pad_to_mask_clearance: 0.125 -> 0.01
