File: KiCad/Generic0.kicad_pcb (KiCad board)
At the start: 2 copper layers, 13.2 x 13.5 mm, 9 parts, among them J1 Shelly, U1 ESP32-PICO-MINI-02

Commit message: Tweak
Routing:
- net GND: track 3.91 -> 7.69 mm, vias 4 -> 3
- net TX: track 8.93 -> 10.1 mm
- net RX: track 8.74 -> 8.10 mm
Other:
- board text added: "RGB: 22/19/7"
- board text removed: "22/19/7"
