File: KiCad/USBA.kicad_sch (KiCad schematic)
At the start: 18 parts, among them J1 USB_A, J2 Shelly, U1 ESP32-PICO-MINI-02, U2 LMR16006+FB, U4 QR

Commit message: PCB make
Parts:
- added C5: 10nF, RevK:C_0603, symbol Device:C
- R6: footprint (none) -> RevK:R_0603
Connections:
- net EN: now also C5.2
- net GND: now also C5.1
Other:
- moved on the sheet: R6
Changed lines of the file:
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@@
   (junction (at 125.095 60.325) (diameter 0) (color 0 0 0 0)
   )
+  (junction (at 81.915 51.435) (diameter 0) (color 0 0 0 0)
+  )
   (junction (at 125.095 55.245) (diameter 0) (color 0 0 0 0)
-  )
-  (junction (at 92.71 51.435) (diameter 0) (color 0 0 0 0)
   )
   (junction (at 164.465 107.315) (diameter 0) (color 0 0 0 0)
@@
   (no_connect (at 125.095 89.535))
   (no_connect (at 94.615 84.455))
+  (no_connect (at 94.615 53.975))
   (no_connect (at 94.615 61.595))
   (no_connect (at 94.615 64.135))
   (no_connect (at 94.615 66.675))
-  (no_connect (at 94.615 53.975))
   (no_connect (at 94.615 81.915))
   (no_connect (at 125.095 86.995))
@@
     (stroke (width 0) (type default) (color 0 0 0 0))
   )
-  (wire (pts (xy 92.71 51.435) (xy 94.615 51.435))
-    (stroke (width 0) (type default) (color 0 0 0 0))
-  )
   (wire (pts (xy 158.115 97.155) (xy 164.465 97.155))
     (stroke (width 0) (type default) (color 0 0 0 0))
@@
     (stroke (width 0) (type default) (color 0 0 0 0))
   )
+  (wire (pts (xy 81.915 51.435) (xy 94.615 51.435))
+    (stroke (width 0) (type default) (color 0 0 0 0))
+  )
+  (wire (pts (xy 75.565 51.435) (xy 81.915 51.435))
+    (stroke (width 0) (type default) (color 0 0 0 0))
+  )
   (wire (pts (xy 153.67 98.425) (xy 158.115 98.425))
     (stroke (width 0) (type default) (color 0 0 0 0))
@@
   )
   (wire (pts (xy 125.095 55.245) (xy 127 55.245))
-    (stroke (width 0) (type default) (color 0 0 0 0))
-  )
-  (wire (pts (xy 89.535 51.435) (xy 92.71 51.435))
     (stroke (width 0) (type default) (color 0 0 0 0))
   )
@@
     )
   )
-  (global_label "EN" (shape input) (at 89.535 51.435 180) (fields_autoplaced)
+  (global_label "EN" (shape input) (at 75.565 51.435 180) (fields_autoplaced)
     (effects (font (size 1.27 1.27)) (justify right))
-    (property "Intersheet References" "${INTERSHEET_REFS}" (id 0) (at 39.37 14.605 0)
+    (property "Intersheet References" "${INTERSHEET_REFS}" (id 0) (at 25.4 14.605 0)
       (effects (font (size 1.27 1.27)) hide)
     )
@@
     (pin "~")
   )
-  (symbol (lib_id "Device:R") (at 92.71 47.625 0) (unit 1)
-    (in_bom yes) (on_board yes)
-    (property "Reference" "R6" (id 0) (at 94.488 46.7903 0)
-      (effects (font (size 1.27 1.27)) (justify left))
-    )
-    (property "Value" "10k" (id 1) (at 92.71 48.895 90)
-      (effects (font (size 1.27 1.27)) (justify left))
-    )
-    (property "Footprint" "" (id 2) (at 90.932 47.625 90)
-      (effects (font (size 1.27 1.27)) hide)
-    )
-    (property "Datasheet" "~" (id 3) (at 92.71 47.625 0)
-      (effects (font (size 1.27 1.27)) hide)
-    )
-    (pin "1")
-    (pin "2")
-  )
-  (symbol (lib_id "power:+3.3V") (at 92.71 43.815 0) (unit 1)
+  (symbol (lib_id "Device:R") (at 81.915 47.625 0) (unit 1)
+    (in_bom yes) (on_board yes)
+    (property "Reference" "R6" (id 0) (at 83.693 46.7903 0)
+      (effects (font (size 1.27 1.27)) (justify left))
+    )
+    (property "Value" "10k" (id 1) (at 81.915 48.895 90)
+      (effects (font (size 1.27 1.27)) (justify left))
+    )
+    (property "Footprint" "RevK:R_0603" (id 2) (at 80.137 47.625 90)
+      (effects (font (size 1.27 1.27)) hide)
+    )
+    (property "Datasheet" "~" (id 3) (at 81.915 47.625 0)
+      (effects (font (size 1.27 1.27)) hide)
+    )
+    (pin "1")
+    (pin "2")
+  )
+  (symbol (lib_id "power:+3.3V") (at 81.915 43.815 0) (unit 1)
     (in_bom yes) (on_board yes) (fields_autoplaced)
-    (property "Reference" "#PWR0103" (id 0) (at 92.71 47.625 0)
-      (effects (font (size 1.27 1.27)) hide)
-    )
-    (property "Value" "+3.3V" (id 1) (at 92.71 40.2392 0))
-    (property "Footprint" "" (id 2) (at 92.71 43.815 0)
-      (effects (font (size 1.27 1.27)) hide)
-    )
-    (property "Datasheet" "" (id 3) (at 92.71 43.815 0)
+    (property "Reference" "#PWR0103" (id 0) (at 81.915 47.625 0)
+      (effects (font (size 1.27 1.27)) hide)
+    )
+    (property "Value" "+3.3V" (id 1) (at 81.915 40.2392 0))
+    (property "Footprint" "" (id 2) (at 81.915 43.815 0)
+      (effects (font (size 1.27 1.27)) hide)
+    )
+    (property "Datasheet" "" (id 3) (at 81.915 43.815 0)
       (effects (font (size 1.27 1.27)) hide)
     )
@@
     (pin "1")
   )
+  (symbol (lib_id "Device:C") (at 81.915 55.245 180) (unit 1)
+    (in_bom yes) (on_board yes) (fields_autoplaced)
+    (property "Reference" "C5" (id 0) (at 84.836 54.4103 0)
+      (effects (font (size 1.27 1.27)) (justify right))
+    )
+    (property "Value" "10nF" (id 1) (at 84.836 56.9472 0)
+      (effects (font (size 1.27 1.27)) (justify right))
+    )
+    (property "Footprint" "RevK:C_0603" (id 2) (at 80.9498 51.435 0)
+      (effects (font (size 1.27 1.27)) hide)
+    )
+    (property "Datasheet" "~" (id 3) (at 81.915 55.245 0)
+      (effects (font (size 1.27 1.27)) hide)
+    )
+    (property "Part No" "0603-10nF-50V" (id 4) (at 81.915 55.245 90)
+      (effects (font (size 1.27 1.27)) hide)
+    )
+    (pin "1")
+    (pin "2")
+  )
   (symbol (lib_id "Device:C") (at 217.805 103.505 0) (unit 1)
     (in_bom yes) (on_board yes) (fields_autoplaced)
@@
     (pin "2")
   )
+  (symbol (lib_id "power:GND") (at 81.915 59.055 0) (unit 1)
+    (in_bom yes) (on_board yes) (fields_autoplaced)
+    (property "Reference" "#PWR0110" (id 0) (at 81.915 65.405 0)
+      (effects (font (size 1.27 1.27)) hide)
+    )
+    (property "Value" "GND" (id 1) (at 81.915 63.4984 0))
+    (property "Footprint" "" (id 2) (at 81.915 59.055 0)
+      (effects (font (size 1.27 1.27)) hide)
+    )
+    (property "Datasheet" "" (id 3) (at 81.915 59.055 0)
+      (effects (font (size 1.27 1.27)) hide)
+    )
+    (pin "1")
+  )
   (symbol (lib_id "power:+3.3V") (at 127.635 60.325 270) (unit 1)
     (in_bom yes) (on_board yes)
@@
       (reference "#PWR0109") (unit 1) (value "VBUS") (footprint "")
     )
+    (path "/db389fa8-d679-470a-8df6-c46c5aa5eb66"
+      (reference "#PWR0110") (unit 1) (value "GND") (footprint "")
+    )
     (path "/77370c6e-b467-4079-90f2-37fc34a6b23c"
       (reference "C1") (unit 1) (value "0.1uF") (footprint "RevK:C_0603_")
@@
       (reference "C4") (unit 1) (value "100nF") (footprint "RevK:C_0603")
     )
+    (path "/b51431db-2560-4de9-83f6-1c1814dc0cbf"
+      (reference "C5") (unit 1) (value "10nF") (footprint "RevK:C_0603")
+    )
     (path "/00000000-0000-0000-0000-000060cf36bc"
       (reference "D1") (unit 1) (value "RGB") (footprint "RevK:LED-RGB-1.6x1.6")
@@
     )
     (path "/550905cb-407f-443f-a9fb-9ce7295efa67"
-      (reference "R6") (unit 1) (value "10k") (footprint "")
+      (reference "R6") (unit 1) (value "10k") (footprint "RevK:R_0603")
     )
     (path "/7a10be77-a011-4709-ad8a-7ab46326680b"
