File: PCB/Generic5/Generic5.kicad_pcb (KiCad board)
At the start: 2 copper layers, 12.5 x 31 mm, 29 parts, among them J1 Conn_01x04, J2 USB-C, Q1 PMF170XP,115, U1 ESP32-PICO-MINI-02, U2 FT231XQ, U3 LMR16006+FB

Commit message: New LED Generic 5
Parts:
- removed D3: Schottky, RevK:Hidden
- removed JP1, JP2: Jumper_2_Open, RevK:Pad_0603_Open
- removed JP3: Jumper_2_Bridged, RevK:Pad_0603_Bridged
- added Q2: PMF250XNEX, RevK:SOT-323_SC-70, B.Cu at (103.0, 84.8)
- C2: value 0.1uF -> 100nF; footprint RevK:Hidden -> RevK:C_0603_
- C3, C4: footprint RevK:Hidden -> RevK:C_0805_
- D1: value D -> LED_BARG; footprint RevK:D_1206 -> RevK:MHS190RGBCT
- D2: value RGB -> Schottky; footprint RevK:LED-RGB-1.6x1.6 -> RevK:D_1206_
- J1: value Conn_01x04 -> Conn_01x03; footprint RevK:Molex_MiniSPOX_H4RA -> RevK:PTSM-HH-3-RA
- J2: footprint RevK:USC16-TR-Round -> RevK:USC16-TR-PTH
- L1: footprint RevK:Hidden -> RevK:L_4x4_
- Q1: footprint Package_TO_SOT_SMD:SOT-323_SC-70 -> RevK:SOT-323_SC-70
- R10: value 30k 1% or NF -> 30k 1%
- R2: value 680R -> 300R
- R3: value 2K -> 1K
- R4: value 220R -> 100R
- R9: value 100k 1% or 0R -> 100k 1%
- U3: value LMR16006+FB -> LMR16006XDDCR; footprint RevK:RegulatorBlockFB -> RevK:SOT-23-Thin-6-Reg
- moved D2 100.3 mm to (98.1, 107.0)
- moved R4 84.5 mm to (97.9, 82.0), turned to 0 degrees
- moved R3 84.0 mm to (97.9, 85.0)
- moved R2 83.8 mm to (97.9, 83.5)
- moved D1 81.1 mm to (95.8, 83.5), turned to -90 degrees
- moved C1 80.9 mm to (96.2, 94.5)
- moved C2 80.9 mm to (101.0, 111.4)
- moved L1 80.9 mm to (101.2, 105.4)
- moved R10 80.9 mm to (103.0, 99.8)
- moved R11 80.9 mm to (95.0, 99.8)
- moved R12 80.9 mm to (95.0, 96.9)
- moved R5 80.9 mm to (96.2, 99.8)
- moved R6 80.9 mm to (101.8, 99.8)
- moved R7 80.9 mm to (99.2, 99.8)
- moved R8 80.9 mm to (100.5, 99.8)
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Connections:
- D1 pad 1: IO3 -> Net-(D1-Pad1)
- D1 pad 2: GND -> +3V3
- J1 pad 1: IO1 -> GND
- J1 pad 3: IO3 -> VBUS
- Q1 pad 1: FET -> LED
- Q1 pad 2: +3V3 -> VBUS
- Q1 pad 3: IO3 -> Net-(J1-Pad2)
- R2 pad 1: Net-(D2-Pad2) -> Net-(D1-Pad3)
- R3 pad 1: Net-(D2-Pad3) -> Net-(D1-Pad4)
- R4 pad 1: Net-(D2-Pad4) -> Net-(D1-Pad1)
- U1 pad 18: FET -> unconnected-(U1-Pad18)
- U1 pad 24: B -> unconnected-(U1-Pad24)
- U1 pad 26: R -> LED
- U1 pad 27: IO1 -> unconnected-(U1-Pad27)
- U1 pad 28: G -> unconnected-(U1-Pad28)
- U1 pad 33: IO3 -> R
- U1 pad 34: IO2 -> G
- U1 pad 35: IO4 -> B
- U3 pad 1: VBUS -> unconnected-(U3-Pad1)
- U3 pad 2: VBUS -> GND
- U3 pad 3: GND -> Net-(R10-Pad2)
- U3 pad 4: +3V3 -> VBUS
- U3 pad 5: Net-(R10-Pad2) -> VBUS
Routing:
- net VBUS: track 69.2 -> 82.9 mm
- net EN: track 26.1 -> 13.0 mm
- net FET: track 11.1 -> 0.00 mm, vias 1 -> 0
- net LED: track 0.00 -> 11.0 mm, vias 0 -> 1
- net IO3: track 9.14 -> 0.00 mm
- net GND: track 62.7 -> 69.8 mm, vias 8 -> 6
- net IO2: track 6.19 -> 0.00 mm, vias 1 -> 0
- net Net-(J1-Pad2): track 3.40 -> 9.45 mm
- net G: track 7.89 -> 13.5 mm
- net Net-(D2-Pad4): track 5.27 -> 0.00 mm
- net IO1: track 4.37 -> 0.00 mm
- net Net-(D2-Pad2): track 2.86 -> 0.00 mm
- net R: track 11.2 -> 8.36 mm
- net IO4: track 2.24 -> 0.00 mm
- net Net-(D1-Pad4): track 0.00 -> 1.89 mm
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Other:
- board size 12.5 x 31 mm -> 11.5 x 31.5 mm
- board text added: "Generic5 - LED"
- board text removed: "14"
- board text removed: "19"
- board text removed: "21"
- board text removed: "22"
- board text removed: "5V"
- board text removed: "7"
- board text removed: "Generic5"
- board text removed: "⏚"
