File: PCB/LED/LED.kicad_sch (KiCad schematic)
At the start: 26 parts, among them J1 Conn_01x03, J2 USB-C, Q1 PMF170XP,115, Q2 PMF250XNEX, U1 ESP32-PICO-MINI-02, U2 FT231XQ, U3 LMR16006XDDCR

Commit message: New
Parts:
- removed C1: 100nF, RevK:C_0603, symbol Device:C
- removed R11: 4k7, RevK:R_0603, symbol Device:R
- removed R12: 10k, RevK:R_0603, symbol Device:R
- removed R7, R8: 27R, RevK:R_0603, symbol Device:R
- removed U2: FT231XQ, RevK:QFN-20-1EP_4x4mm_P0.5mm_EP2.5x2.5mm, symbol RevK:FT231XQ
- added J3: Shelly, RevK:Shelly, symbol RevK:Shelly
- added U2: QR, RevK:QR-LED, symbol RevK:QR
- J2: footprint RevK:USC16-TR-PTH -> RevK:USC16-TR
Connections:
- net +3V3: now also J3.3 (3V3)
- net G: now also U1.28 (IO8); no longer U1.34 (IO22)
- net GND: now also U1.33 (IO19), J3.1 (GND)
- net GPIO0: now also J3.2 (0)
- net I: now also J3.4 (Rx)
- net LED: now also U1.34 (IO22); no longer U1.26 (IO20)
- net O: now also J3.5 (Tx)
- net R: now also U1.26 (IO20); no longer U1.33 (IO19)
- no-connect marks 19 -> 21
Other:
- title: Generic ESP32-PICO-MINI module -> LED driver
- moved on the sheet: J1, Q1, Q2

Commit message: Library update
Parts:
- J2: LCSC Part # (none) -> C709357; Manufacturer Valcon -> (none); Order URL https://www.toby.co.uk/signal-to-board-connectors/usb-conne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 -> (none); Part No CSP-USC16-TR -> (none)
Changed lines of the file:
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@@
       (effects (font (size 1.27 1.27)) hide)
     )
-    (property "Manufacturer" "Valcon" (id 4) (at 157.48 40.64 0)
+    (property "LCSC Part #" "C709357" (id 4) (at 157.48 40.64 0)
       (effects (font (size 1.27 1.27)) hide)
     )
-    (property "Part No" "CSP-USC16-TR" (id 5) (at 157.48 40.64 0)
-      (effects (font (size 1.27 1.27)) hide)
-    )
-    (property "Order URL" "https://www.toby.co.uk/signal-to-board-connectors/usb-connectors/csp-usc16-tr-valcon-usb-type-c-surface-mount-pcb-socket/" (id 6) (at 157.48 40.64 0)
-      (effects (font (size 1.27 1.27)) hide)
-    )

Commit message: New PCB
Parts:
- J2: JLCPCB Rotation Offset (none) -> 180
- U3: JLCPCB Rotation Offset 90 -> 180; LCSC Part # C87080 -> C290195
Changed lines of the file:
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@@
+      (effects (font (size 1.27 1.27)) hide)
+    )
+    (property "JLCPCB Rotation Offset" "180" (id 5) (at 157.48 40.64 0)
       (effects (font (size 1.27 1.27)) hide)
     )
@@
       (effects (font (size 1.27 1.27)) hide)
     )
-    (property "LCSC Part #" "C87080" (id 6) (at 236.22 51.435 0)
-      (effects (font (size 1.27 1.27)) hide)
-    )
-    (property "JLCPCB Rotation Offset" "90" (id 7) (at 260.985 51.435 0)
-      (effects (font (size 1.27 1.27)) hide)
-    )
+    (property "LCSC Part #" "C290195" (id 6) (at 236.22 51.435 0)
+      (effects (font (size 1.27 1.27)) hide)
+    )
+    (property "JLCPCB Rotation Offset" "180" (id 7) (at 260.985 51.435 0)
+      (effects (font (size 1.27 1.27)) hide)
+    )
