File: PCB/USBA2/USBA2.kicad_sch (KiCad schematic)
At the start: 20 parts, among them J1 USB_A, U1 ESP32-PICO-MINI-02, U2 LMR16006YDDCR, U3 CH340X, U4 QR

Commit message: Rotation fixes
Parts:
- D2: JLCPCB Rotation Offset 0 -> (none)
- U1: JLCPCB Rotation Offset 180 -> (none)
Changed lines of the file:
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@@
-      (effects (font (size 1.27 1.27)) hide)
-    )
-    (property "JLCPCB Rotation Offset" "180" (at 106.68 72.39 0)
       (effects (font (size 1.27 1.27)) hide)
     )
@@
       (effects (font (size 1.27 1.27)) hide)
     )
-    (property "JLCPCB Rotation Offset" "0" (at 185.42 106.68 0)
-      (effects (font (size 1.27 1.27)) hide)
-    )
