File: PCB/USBA3/USBA.kicad_sch (KiCad schematic)
At the start: 29 parts, among them J1 USB_A, U1 ESP32-PICO-MINI-02, U2 Barcode, U3 CH340X, U4 QR, U5 MD8942

Commit message: Better rails
Parts:
- removed FID1, FID2, FID3, FID4, FID5, FID6, FID7, FID8: Fiducial, Fiducial:Fiducial_1mm_Mask2mm, symbol Mechanical:Fiducial
- added PCB1: 70x70, RevK:PCB7070, symbol RevK:PCB
Changed lines of the file:
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@@
-    )
-  )
-  (symbol (lib_id "Mechanical:Fiducial") (at 257.175 150.495 0) (unit 1)
-    (in_bom no) (on_board yes) (dnp no) (fields_autoplaced)
-    (property "Reference" "FID2" (at 259.334 149.471 0)
-      (effects (font (size 1.27 1.27)) (justify left))
-    )
-    (property "Value" "Fiducial" (at 259.334 151.519 0)
-      (effects (font (size 1.27 1.27)) (justify left))
-    )
-    (property "Footprint" "Fiducial:Fiducial_1mm_Mask2mm" (at 257.175 150.495 0)
-      (effects (font (size 1.27 1.27)) hide)
-    )
-    (property "Datasheet" "~" (at 257.175 150.495 0)
-      (effects (font (size 1.27 1.27)) hide)
-    )
-    (instances
-      (project "USBA"
-        (path "/2d210a96-f81f-42a9-8bf4-1b43c11086f3"
-          (reference "FID2") (unit 1)
-        )
-      )
-      (project "Faikin"
-        (path "/46c350bb-7de4-4e81-aafd-4af55e37aab0"
-          (reference "FID6") (unit 1)
-        )
-      )
-    )
-  )
-  (symbol (lib_id "Mechanical:Fiducial") (at 257.175 155.575 0) (unit 1)
-    (in_bom no) (on_board yes) (dnp no) (fields_autoplaced)
-    (property "Reference" "FID3" (at 259.334 154.551 0)
-      (effects (font (size 1.27 1.27)) (justify left))
-    )
-    (property "Value" "Fiducial" (at 259.334 156.599 0)
-      (effects (font (size 1.27 1.27)) (justify left))
-    )
-    (property "Footprint" "Fiducial:Fiducial_1mm_Mask2mm" (at 257.175 155.575 0)
-      (effects (font (size 1.27 1.27)) hide)
-    )
-    (property "Datasheet" "~" (at 257.175 155.575 0)
-      (effects (font (size 1.27 1.27)) hide)
-    )
-    (instances
-      (project "USBA"
-        (path "/2d210a96-f81f-42a9-8bf4-1b43c11086f3"
-          (reference "FID3") (unit 1)
-        )
-      )
-      (project "Faikin"
-        (path "/46c350bb-7de4-4e81-aafd-4af55e37aab0"
-          (reference "FID7") (unit 1)
-        )
-      )
     )
   )
@@
         (path "/babeabf2-f3b0-4ed5-8d9e-0215947e6cf3"
           (reference "#PWR024") (unit 1)
-        )
-      )
-    )
-  )
-  (symbol (lib_id "Mechanical:Fiducial") (at 269.24 155.575 0) (unit 1)
-    (in_bom no) (on_board yes) (dnp no) (fields_autoplaced)
-    (property "Reference" "FID7" (at 271.399 154.551 0)
-      (effects (font (size 1.27 1.27)) (justify left))
-    )
-    (property "Value" "Fiducial" (at 271.399 156.599 0)
-      (effects (font (size 1.27 1.27)) (justify left))
-    )
-    (property "Footprint" "Fiducial:Fiducial_1mm_Mask2mm" (at 269.24 155.575 0)
-      (effects (font (size 1.27 1.27)) hide)
-    )
-    (property "Datasheet" "~" (at 269.24 155.575 0)
-      (effects (font (size 1.27 1.27)) hide)
-    )
-    (instances
-      (project "USBA"
-        (path "/2d210a96-f81f-42a9-8bf4-1b43c11086f3"
-          (reference "FID7") (unit 1)
-        )
-      )
-      (project "Faikin"
-        (path "/46c350bb-7de4-4e81-aafd-4af55e37aab0"
-          (reference "FID3") (unit 1)
         )
       )
@@
         (path "/2d210a96-f81f-42a9-8bf4-1b43c11086f3"
           (reference "#PWR0102") (unit 1)
-        )
-      )
-    )
-  )
-  (symbol (lib_id "Mechanical:Fiducial") (at 269.24 150.495 0) (unit 1)
-    (in_bom no) (on_board yes) (dnp no) (fields_autoplaced)
-    (property "Reference" "FID6" (at 271.399 149.471 0)
-      (effects (font (size 1.27 1.27)) (justify left))
-    )
-    (property "Value" "Fiducial" (at 271.399 151.519 0)
-      (effects (font (size 1.27 1.27)) (justify left))
-    )
-    (property "Footprint" "Fiducial:Fiducial_1mm_Mask2mm" (at 269.24 150.495 0)
-      (effects (font (size 1.27 1.27)) hide)
-    )
-    (property "Datasheet" "~" (at 269.24 150.495 0)
-      (effects (font (size 1.27 1.27)) hide)
-    )
-    (instances
-      (project "USBA"
-        (path "/2d210a96-f81f-42a9-8bf4-1b43c11086f3"
-          (reference "FID6") (unit 1)
-        )
-      )
-      (project "Faikin"
-        (path "/46c350bb-7de4-4e81-aafd-4af55e37aab0"
-          (reference "FID2") (unit 1)
         )
       )
@@
     )
   )
+  (symbol (lib_id "RevK:PCB") (at 250.19 172.72 0) (unit 1)
+    (in_bom no) (on_board yes) (dnp no)
+    (property "Reference" "PCB1" (at 250.19 182.88 0)
+      (effects (font (size 1.27 1.27)) hide)
+    )
+    (property "Value" "70x70" (at 250.19 172.72 0)
+      (effects (font (size 1.27 1.27)))
+    )
+    (property "Footprint" "RevK:PCB7070" (at 250.19 167.005 0)
+      (effects (font (size 1.27 1.27)) hide)
+    )
+    (property "Datasheet" "" (at 250.19 172.72 0)
+      (effects (font (size 1.27 1.27)) hide)
+    )
+    (instances
+      (project "USBA"
+        (path "/2d210a96-f81f-42a9-8bf4-1b43c11086f3"
+          (reference "PCB1") (unit 1)
+        )
+      )
+    )
+  )
   (symbol (lib_id "RevK:Hidden") (at 198.12 127 0) (unit 1)
     (in_bom yes) (on_board yes) (dnp no)
@@
     )
   )
-  (symbol (lib_id "Mechanical:Fiducial") (at 269.24 160.655 0) (unit 1)
-    (in_bom no) (on_board yes) (dnp no) (fields_autoplaced)
-    (property "Reference" "FID8" (at 271.399 159.631 0)
-      (effects (font (size 1.27 1.27)) (justify left))
-    )
-    (property "Value" "Fiducial" (at 271.399 161.679 0)
-      (effects (font (size 1.27 1.27)) (justify left))
-    )
-    (property "Footprint" "Fiducial:Fiducial_1mm_Mask2mm" (at 269.24 160.655 0)
-      (effects (font (size 1.27 1.27)) hide)
-    )
-    (property "Datasheet" "~" (at 269.24 160.655 0)
-      (effects (font (size 1.27 1.27)) hide)
-    )
-    (instances
-      (project "USBA"
-        (path "/2d210a96-f81f-42a9-8bf4-1b43c11086f3"
-          (reference "FID8") (unit 1)
-        )
-      )
-      (project "Faikin"
-        (path "/46c350bb-7de4-4e81-aafd-4af55e37aab0"
-          (reference "FID4") (unit 1)
-        )
-      )
-    )
-  )
   (symbol (lib_id "RevK:Barcode") (at 271.145 172.085 0) (unit 1)
     (in_bom no) (on_board yes) (dnp no) (fields_autoplaced)
@@
     )
   )
-  (symbol (lib_id "Mechanical:Fiducial") (at 257.175 160.655 0) (unit 1)
-    (in_bom no) (on_board yes) (dnp no) (fields_autoplaced)
-    (property "Reference" "FID4" (at 259.334 159.631 0)
-      (effects (font (size 1.27 1.27)) (justify left))
-    )
-    (property "Value" "Fiducial" (at 259.334 161.679 0)
-      (effects (font (size 1.27 1.27)) (justify left))
-    )
-    (property "Footprint" "Fiducial:Fiducial_1mm_Mask2mm" (at 257.175 160.655 0)
-      (effects (font (size 1.27 1.27)) hide)
-    )
-    (property "Datasheet" "~" (at 257.175 160.655 0)
-      (effects (font (size 1.27 1.27)) hide)
-    )
-    (instances
-      (project "USBA"
-        (path "/2d210a96-f81f-42a9-8bf4-1b43c11086f3"
-          (reference "FID4") (unit 1)
-        )
-      )
-      (project "Faikin"
-        (path "/46c350bb-7de4-4e81-aafd-4af55e37aab0"
-          (reference "FID8") (unit 1)
-        )
-      )
-    )
-  )
   (symbol (lib_id "Device:C") (at 78.74 53.34 180) (unit 1)
     (in_bom yes) (on_board yes) (dnp no) (fields_autoplaced)
@@
     )
   )
-  (symbol (lib_id "Mechanical:Fiducial") (at 269.24 145.415 0) (unit 1)
-    (in_bom no) (on_board yes) (dnp no) (fields_autoplaced)
-    (property "Reference" "FID5" (at 271.399 144.391 0)
-      (effects (font (size 1.27 1.27)) (justify left))
-    )
-    (property "Value" "Fiducial" (at 271.399 146.439 0)
-      (effects (font (size 1.27 1.27)) (justify left))
-    )
-    (property "Footprint" "Fiducial:Fiducial_1mm_Mask2mm" (at 269.24 145.415 0)
-      (effects (font (size 1.27 1.27)) hide)
-    )
-    (property "Datasheet" "~" (at 269.24 145.415 0)
-      (effects (font (size 1.27 1.27)) hide)
-    )
-    (instances
-      (project "USBA"
-        (path "/2d210a96-f81f-42a9-8bf4-1b43c11086f3"
-          (reference "FID5") (unit 1)
-        )
-      )
-      (project "Faikin"
-        (path "/46c350bb-7de4-4e81-aafd-4af55e37aab0"
-          (reference "FID1") (unit 1)
-        )
-      )
-    )
-  )
   (symbol (lib_id "RevK:Hidden") (at 198.12 128.905 270) (unit 1)
     (in_bom yes) (on_board yes) (dnp no)
@@
         )
       )
-    )
-  )
-  (symbol (lib_id "Mechanical:Fiducial") (at 257.175 145.415 0) (unit 1)
-    (in_bom no) (on_board yes) (dnp no) (fields_autoplaced)
-    (property "Reference" "FID1" (at 259.334 144.391 0)
-      (effects (font (size 1.27 1.27)) (justify left))
-    )
-    (property "Value" "Fiducial" (at 259.334 146.439 0)
-      (effects (font (size 1.27 1.27)) (justify left))
-    )
-    (property "Footprint" "Fiducial:Fiducial_1mm_Mask2mm" (at 257.175 145.415 0)
-      (effects (font (size 1.27 1.27)) hide)
-    )
-    (property "Datasheet" "~" (at 257.175 145.415 0)
-      (effects (font (size 1.27 1.27)) hide)
-    )
-    (instances
-      (project "USBA"
-        (path "/2d210a96-f81f-42a9-8bf4-1b43c11086f3"
-          (reference "FID1") (unit 1)
-        )
-      )
-      (project "Faikin"
-        (path "/46c350bb-7de4-4e81-aafd-4af55e37aab0"
-          (reference "FID5") (unit 1)
-        )
-      )
