File: PCB/Generic/Generic.kicad_pcb (KiCad board)
At the start: 2 copper layers, 19 x 29 mm, 39 parts, among them J1 Connector, J2 USB-C, J3 DC, U1 ESP32-WROOM-32, U2 FT231XQ, U3 LMR16006+FB

Commit message: More tidy
Parts:
- C6: value 0.1uF -> 100nF; footprint RevK:Hidden -> RevK:C_0603_
- C7, C8: footprint RevK:Hidden -> RevK:C_0805_
- D1: value RGB -> LED_BARG; footprint RevK:LED-RGB-1.6x1.6 -> RevK:MHS190RGBCT
- D5: footprint RevK:Hidden -> RevK:D_1206_
- J1: footprint RevK:Molex_MiniSPOX_H6RA -> RevK:PTSM-HH-6-RA
- J2: footprint RevK:USC16-TR-Round -> RevK:USC16-TR
- L1: footprint RevK:Hidden -> RevK:L_4x4_
- R10: value 220R -> 100R
- R17: value 100k 1% or 0R -> 100k 1%
- R18: value 30k 1% or NF -> 30k 1%
- R8: value 680R -> 300R
- R9: value 2K -> 1K
- U3: value LMR16006+FB -> LMR16006XDDCR; footprint RevK:RegulatorBlockFB -> RevK:SOT-23-Thin-6-Reg
- moved J2 4.44 mm to (131.8, 111.1)
- moved D1 0.81 mm to (118.4, 99.8)
- moved J1 0.14 mm to (126.7, 120.4)
- moved C3 0.08 mm to (132.8, 117.5)
- moved C4 0.08 mm to (131.6, 117.5)
Connections:
- D1 pad 1: +3V3 -> Net-(D1-Pad1)
- D1 pad 2: Net-(D1-Pad2) -> +3V3
- R10 pad 1: Net-(D1-Pad4) -> Net-(D1-Pad1)
- R8 pad 1: Net-(D1-Pad2) -> Net-(D1-Pad3)
- R9 pad 1: Net-(D1-Pad3) -> Net-(D1-Pad4)
- U3 pad 1: DC -> unconnected-(U3-Pad1)
- U3 pad 2: DC -> GND
- U3 pad 3: GND -> Net-(R17-Pad2)
- U3 pad 4: +3V3 -> DC
- U3 pad 5: Net-(R17-Pad2) -> DC
Routing:
- net GND: track 129.8 -> 136.2 mm
- net Net-(D1-Pad3): track 5.49 -> 1.53 mm
- net Net-(D1-Pad1): track 0.00 -> 3.14 mm
- net +3V3: track 112.2 -> 115.0 mm
- net Net-(D1-Pad2): track 1.02 -> 0.00 mm
- net IO4: track 28.2 -> 27.5 mm

Commit message: PCB Update
Connections:
- J1 pad 6: Net-(J1-Pad6) -> Net-(J1-Pin_6)
- J2 pad A5: Net-(J2-PadA5) -> Net-(J2-CC1)
- J2 pad B5: Net-(J2-PadB5) -> Net-(J2-CC2)
- U2 pad 16: Net-(R15-Pad2) -> Net-(U2-CBUS3)
- U3 pad 3: Net-(R17-Pad2) -> Net-(U3-FB)
