File: PCB/Generic/Generic.kicad_sch (KiCad schematic)
At the start: 39 parts, among them J1 Connector, J2 USB-C, J3 DC, U1 ESP32-WROOM-32, U2 FT231XQ, U3 LMR16006+FB

Commit message: More tidy
Parts:
- removed D1: RGB, RevK:LED-RGB-1.6x1.6, symbol Device:LED_ARGB
- removed U3: LMR16006+FB, RevK:RegulatorBlockFB, symbol RevK:LMR16006+FB
- added D1: LED_BARG, RevK:MHS190RGBCT, symbol Device:LED_BARG
- added U3: LMR16006XDDCR, RevK:SOT-23-Thin-6-Reg, symbol RevK:LMR16006XDDCR
- C6: value 0.1uF -> 100nF; footprint RevK:Hidden -> RevK:C_0603_; LCSC Part # (none) -> C30926
- C7: footprint RevK:Hidden -> RevK:C_0805_; LCSC Part # (none) -> C19110; Note 0603 or 0805 -> (none)
- C8: footprint RevK:Hidden -> RevK:C_0805_; LCSC Part # (none) -> C17024; Note 0603 or 0805 -> (none)
- D5: footprint RevK:Hidden -> RevK:D_1206_; JLCPCB Rotation Offset (none) -> 0; LCSC Part # (none) -> C143805; Part No CD1206-B2100 -> (none)
- J1: footprint RevK:Molex_MiniSPOX_H6RA -> RevK:PTSM-HH-6-RA; Manufacturer Molex -> (none); Notes Not fitted -> (none); Part No 0022057065 -> (none)
- J2: footprint RevK:USC16-TR-Round -> RevK:USC16-TR
- J3: now left out of the parts list
- L1: footprint RevK:Hidden -> RevK:L_4x4_; LCSC Part # (none) -> C354575; Manufacturer Laird -> (none); Part No TYA4020 -> (none)
- R10: value 220R -> 100R; Part No (none) -> 0603-220R
- R17: value 100k 1% or 0R -> 100k 1%; LCSC Part # (none) -> C14675
- R18: value 30k 1% or NF -> 30k 1%; LCSC Part # (none) -> C100001
- R8: value 680R -> 300R; Part No (none) -> 0603-680R
- R9: value 2K -> 1K; Part No (none) -> 0603-2K
Connections:
- net +3V3: now also D1.2 (A), U3.7 (VOUT)
- net DC: now also U3.4 (SHDN), U3.5 (VIN)
- net GND: now also U3.2 (GND)
- net at R10.1: now also D1.1 (BK)
- net at R8.1: now also D1.3 (RK)
- net at R9.1: now also D1.4 (GK)
- net at R17.2, R18.2: now also U3.3 (FB)

Commit message: PCB Update
Parts:
- C1, R2, R3, R4, R5, R6, R7: footprint RevK:Pad_1206_0805_Open -> (none); Notes Not fitted -> (none)
- C2, C3, C4, C5: footprint RevK:C_0603 -> (none)
- C6: footprint RevK:C_0603_ -> (none); LCSC Part # C30926 -> (none); Note X7R or X5R 0603 -> (none)
- C7: footprint RevK:C_0805_ -> (none); LCSC Part # C19110 -> (none)
- C8: footprint RevK:C_0805_ -> (none); LCSC Part # C17024 -> (none)
- D1: footprint RevK:MHS190RGBCT -> (none); LCSC Part # C409798 -> (none)
- D2: footprint Diode_SMD:D_1206_3216Metric -> (none)
- D3, D4: Manufacturer Nexperia -> (none); Part No BAV99S -> (none)
- D5: footprint RevK:D_1206_ -> (none); JLCPCB Rotation Offset 0 -> (none); LCSC Part # C143805 -> (none); Manufacturer Bourns -> (none)
- J3: footprint RevK:DC -> (none); Notes Not fitted -> (none)
- L1: footprint RevK:L_4x4_ -> (none); LCSC Part # C354575 -> (none)
- R1, R11, R12, R13, R14, R15, R16: footprint RevK:R_0603 -> (none)
- R10: footprint RevK:R_0603 -> (none); Part No 0603-220R -> (none)
- R17: footprint RevK:R_0603 -> (none); LCSC Part # C14675 -> (none)
- R18: footprint RevK:R_0603 -> (none); LCSC Part # C100001 -> (none)
- R8: footprint RevK:R_0603 -> (none); Part No 0603-680R -> (none)
- R9: footprint RevK:R_0603 -> (none); Part No 0603-2K -> (none)
- U2: MPN (none) -> C132159
- U3: JLCPCB Rotation Offset 90 -> (none); LCSC Part # C87080 -> (none); MPN (none) -> C87080
