File: PCB/Generic0/Generic0.kicad_pcb (KiCad board)
At the start: 2 copper layers, 13.2 x 13.5 mm, 9 parts, among them J1 Shelly, U1 ESP32-PICO-MINI-02

Commit message: Details
Parts:
- moved J1 0.50 mm to (100.0, 50.4)
Routing:
- net GND: track 7.69 -> 5.47 mm
- net TX: track 10.1 -> 9.49 mm
- net +3V3: track 28.6 -> 28.0 mm
Other:
- board size 13.2 x 13.5 mm -> 13.2 x 12.5 mm

Commit message: More tidy
Parts:
- D1: value RGB -> LED_BARG; footprint RevK:LED-RGB-1.6x1.6 -> RevK:MHS190RGBCT
- R1: value 680R -> 300R
- R2: value 2K -> 1K
- R3: value 220R -> 100R
- moved D1 0.42 mm to (104.7, 40.3), turned to 180 degrees
Connections:
- D1 pad 1: +3V3 -> Net-(D1-Pad1)
- D1 pad 2: Net-(D1-Pad2) -> +3V3
- R1 pad 1: Net-(D1-Pad2) -> Net-(D1-Pad3)
- R2 pad 1: Net-(D1-Pad3) -> Net-(D1-Pad4)
- R3 pad 1: Net-(D1-Pad4) -> Net-(D1-Pad1)
Routing:
- net Net-(D1-Pad1): track 0.00 -> 5.52 mm
- net Net-(D1-Pad2): track 5.30 -> 0.00 mm
- net Net-(D1-Pad3): track 1.56 -> 6.85 mm
- net Net-(D1-Pad4): track 5.68 -> 1.64 mm
