File: PCB/Generic0/Generic0.kicad_sch (KiCad schematic)
At the start: 9 parts, among them J1 Shelly, U1 ESP32-PICO-MINI-02

Commit message: More tidy
Parts:
- removed D1: RGB, RevK:LED-RGB-1.6x1.6, symbol Device:LED_ARGB
- added D1: LED_BARG, RevK:MHS190RGBCT, symbol Device:LED_BARG
- R1: value 680R -> 300R; Part No (none) -> 0603-680R
- R2: value 2K -> 1K; Part No (none) -> 0603-2K
- R3: value 220R -> 100R; Part No (none) -> 0603-220R
Connections:
- net +3V3: now also D1.2 (A)
- net at R1.1: now also D1.3 (RK)
- net at R2.1: now also D1.4 (GK)
- net at R3.1: now also D1.1 (BK)

Commit message: PCB Update
Parts:
- D1: LCSC Part # C409798 -> (none); MPN (none) -> C409798
Changed lines of the file:
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@@
       (effects (font (size 1.27 1.27)) hide)
     )
-    (property "LCSC Part #" "C409798" (id 4) (at 71.12 120.65 0)
+    (property "MPN" "C409798" (id 4) (at 71.12 120.65 0)
       (effects (font (size 1.27 1.27)) hide)
     )
