File: PCB/Generic2/Generic2.kicad_pcb (KiCad board)
At the start: 2 copper layers, 35.5 x 22.5 mm, 45 parts, among them J1 Left, J2 Right, J3 USB-C, J4 DC, U1 ESP32-WROOM-32, U2 FT231XQ, U3 LMR16006+FB

Commit message: More tidy
Parts:
- C5: value 0.1uF -> 100nF; footprint RevK:Hidden -> RevK:C_0603_
- C6, C7: footprint RevK:Hidden -> RevK:C_0805_
- D1: value RGB -> LED_BARG; footprint RevK:LED-RGB-1.6x1.6 -> RevK:MHS190RGBCT
- D6: footprint RevK:Hidden -> RevK:D_1206_
- J1, J2: footprint RevK:Molex_MiniSPOX_H8RA -> RevK:PTSM-HH-8-RA
- J3: footprint RevK:USC16-TR-Round -> RevK:USC16-TR
- J4: footprint RevK:PinHeader_1x02_P2.54mm_Vertical -> RevK:DC
- L1: footprint RevK:Hidden -> RevK:L_4x4_
- R11: value 100k 1% or 0R -> 100k 1%
- R12: value 30k 1% or NF -> 30k 1%
- R2: value 680R -> 300R
- R3: value 2K -> 1K
- R4: value 220R -> 100R
- U3: value LMR16006+FB -> LMR16006XDDCR; footprint RevK:RegulatorBlockFB -> RevK:SOT-23-Thin-6-Reg
- moved J3 4.35 mm to (147.7, 105.6)
- moved D1 1.39 mm to (139.4, 89.4), turned to 0 degrees
- turned J4 to -90 degrees
Connections:
- D1 pad 1: +3V3 -> Net-(D1-Pad1)
- D1 pad 2: Net-(D1-Pad2) -> +3V3
- R2 pad 1: Net-(D1-Pad2) -> Net-(D1-Pad3)
- R3 pad 1: Net-(D1-Pad3) -> Net-(D1-Pad4)
- R4 pad 1: Net-(D1-Pad4) -> Net-(D1-Pad1)
- U3 pad 1: DC -> unconnected-(U3-Pad1)
- U3 pad 2: DC -> GND
- U3 pad 3: GND -> Net-(R11-Pad2)
- U3 pad 4: +3V3 -> DC
- U3 pad 5: Net-(R11-Pad2) -> DC
Routing:
- net GND: track 42.0 -> 66.7 mm
- net Net-(D1-Pad1): track 0.00 -> 6.37 mm
- net +3V3: track 119.4 -> 116.2 mm
- net Net-(D1-Pad3): track 5.31 -> 3.06 mm
- net R1: track 17.2 -> 15.9 mm
- net Net-(D1-Pad2): track 1.02 -> 0.00 mm
- net R6: track 8.38 -> 7.56 mm
- net R7: track 5.70 -> 4.89 mm
- net Net-(D1-Pad4): track 4.18 -> 4.94 mm
- net R5: track 5.95 -> 5.22 mm
- net L7: track 16.3 -> 15.8 mm
- net R4: track 8.80 -> 8.27 mm
- net R8: track 12.8 -> 12.3 mm

Commit message: Started some updates, not all complete
Other:
- board text added: "${CURRENT_DATE}"
- board text added: "23/21/22"
- board text added: "3V3"
- board text removed: "${DATE}"
- board text removed: "3.3V"
- board text removed: "RGB: 23/21/22"

Commit message: Messing around, not good
Parts:
- added C8: 1uF, RevK:C_0603, F.Cu at (140.6, 108.1)
- added J5: Shelly, RevK:Shelly, F.Cu at (164.4, 103.9)
- U1: value ESP32-WROOM-32 -> ESP32-PICO-MINI-02; footprint RevK:ESP32-WROOM-32 -> RevK:ESP32-PICO-MINI-02
- moved Logo1 14.8 mm to (169.4, 97.8)
- moved R11 13.2 mm to (155.1, 101.3), turned to 180 degrees
- moved L1 8.49 mm to (151.2, 98.7), turned to 180 degrees
- moved C5 7.51 mm to (157.2, 98.5)
- moved C7 7.26 mm to (149.7, 95.2), turned to -90 degrees
- moved R12 7.04 mm to (155.1, 102.5)
- moved U3 5.46 mm to (153.7, 98.0), turned to 180 degrees
- moved R3 4.26 mm to (139.6, 90.0), turned to 180 degrees
- moved D6 3.57 mm to (152.8, 95.5), turned to 180 degrees
- moved R1 3.20 mm to (140.6, 105.1)
- moved R4 3.04 mm to (139.6, 91.2), turned to 180 degrees
- moved C6 2.66 mm to (155.9, 95.2), turned to -90 degrees
- moved R2 2.47 mm to (139.6, 92.4), turned to 180 degrees
- moved C1 1.70 mm to (141.3, 102.9)
- moved D1 0.84 mm to (139.1, 88.6)
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Connections:
- U1 pad 10: R5 -> unconnected-(U1-I35-Pad10)
- U1 pad 11: R1 -> GND
- U1 pad 12: R6 -> unconnected-(U1-IO32-Pad12)
- U1 pad 13: R2 -> unconnected-(U1-IO33-Pad13)
- U1 pad 14: R7 -> GND
- U1 pad 15: GND -> unconnected-(U1-IO25-Pad15)
- U1 pad 16: R8 -> unconnected-(U1-IO26-Pad16)
- U1 pad 2: +3V3 -> GND
- U1 pad 23: L2 -> GPIO0
- U1 pad 24: L1 -> unconnected-(U1-IO4-Pad24)
- U1 pad 25: GPIO0 -> unconnected-(U1-NC-Pad25)
- U1 pad 26: L3 -> unconnected-(U1-IO20-Pad26)
- U1 pad 27: L7 -> unconnected-(U1-IO7-Pad27)
- U1 pad 28: L4 -> unconnected-(U1-IO8-Pad28)
- U1 pad 29: L6 -> unconnected-(U1-IO5-Pad29)
- U1 pad 3: EN -> +3V3
- U1 pad 30: L5 -> I
- U1 pad 31: L8 -> O
- U1 pad 33: G -> unconnected-(U1-IO19-Pad33)
- U1 pad 34: I -> unconnected-(U1-IO22-Pad34)
- U1 pad 35: O -> unconnected-(U1-IO21-Pad35)
- U1 pad 36: B -> GND
- U1 pad 37: R -> GND
- U1 pad 6: R1 -> unconnected-(U1-I38-Pad6)
- U1 pad 8: R3 -> EN
- U1 pad 9: R4 -> unconnected-(U1-I34-Pad9)
Routing:
- net DC: track 70.5 -> 24.8 mm, vias 4 -> 0
- net GND: track 66.7 -> 26.2 mm, vias 9 -> 2
- net O: track 19.3 -> 51.7 mm, vias 1 -> 2
- net VBUS: track 25.2 -> 52.4 mm, vias 3 -> 2
- net +3V3: track 116.2 -> 91.5 mm, vias 3 -> 5
- net R2: track 21.3 -> 0.00 mm, vias 1 -> 0
- net EN: track 34.2 -> 12.9 mm, vias 1 -> 2
- net R1: track 15.9 -> 2.45 mm
- net L7: track 15.8 -> 2.98 mm
- net G: track 9.86 -> 0.00 mm, vias 1 -> 0
- net L8: track 14.1 -> 5.13 mm, vias 0 -> 1
- net L6: track 13.6 -> 4.98 mm, vias 0 -> 1
- net B: track 8.35 -> 0.00 mm, vias 1 -> 0
- net R8: track 12.3 -> 5.24 mm, vias 0 -> 1
- net Net-(D1-BK): track 6.37 -> 0.00 mm
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