File: PCB/Generic2/Generic2.kicad_sch (KiCad schematic)
At the start: 45 parts, among them J1 Left, J2 Right, J3 USB-C, J4 DC, U1 ESP32-WROOM-32, U2 FT231XQ, U3 LMR16006+FB

Commit message: More tidy
Parts:
- removed D1: RGB, RevK:LED-RGB-1.6x1.6, symbol Device:LED_ARGB
- removed U3: LMR16006+FB, RevK:RegulatorBlockFB, symbol RevK:LMR16006+FB
- added D1: LED_BARG, RevK:MHS190RGBCT, symbol Device:LED_BARG
- added U3: LMR16006XDDCR, RevK:SOT-23-Thin-6-Reg, symbol RevK:LMR16006XDDCR
- C5: value 0.1uF -> 100nF; footprint RevK:Hidden -> RevK:C_0603_; LCSC Part # (none) -> C30926
- C6: footprint RevK:Hidden -> RevK:C_0805_; LCSC Part # (none) -> C19110; Note 0603 or 0805 -> (none)
- C7: footprint RevK:Hidden -> RevK:C_0805_; LCSC Part # (none) -> C17024; Note 0603 or 0805 -> (none)
- D6: footprint RevK:Hidden -> RevK:D_1206_; JLCPCB Rotation Offset (none) -> 0; LCSC Part # (none) -> C143805; Part No CD1206-B2100 -> (none)
- J1, J2: footprint RevK:Molex_MiniSPOX_H8RA -> RevK:PTSM-HH-8-RA
- J3: footprint RevK:USC16-TR-Round -> RevK:USC16-TR
- J4: footprint RevK:PinHeader_1x02_P2.54mm_Vertical -> RevK:DC
- L1: footprint RevK:Hidden -> RevK:L_4x4_; LCSC Part # (none) -> C354575; Manufacturer Laird -> (none); Part No TYA4020 -> (none)
- R11: value 100k 1% or 0R -> 100k 1%; LCSC Part # (none) -> C14675
- R12: value 30k 1% or NF -> 30k 1%; LCSC Part # (none) -> C100001
- R2: value 680R -> 300R; Part No (none) -> 0603-680R
- R3: value 2K -> 1K; Part No (none) -> 0603-2K
- R4: value 220R -> 100R; Part No (none) -> 0603-220R
Connections:
- net +3V3: now also D1.2 (A), U3.7 (VOUT)
- net DC: now also U3.4 (SHDN), U3.5 (VIN)
- net GND: now also U3.2 (GND)
- net at R4.1: now also D1.1 (BK)
- net at R2.1: now also D1.3 (RK)
- net at R3.1: now also D1.4 (GK)
- net at R11.2, R12.2: now also U3.3 (FB)

Commit message: Messing around, not good
Parts:
- removed U1: ESP32-WROOM-32, RevK:ESP32-WROOM-32, symbol RevK:ESP32-WROOM-32
- added C8: 1uF, RevK:C_0603, symbol Device:C
- added J5: Shelly, RevK:Shelly, symbol RevK:Shelly
- added U1: ESP32-PICO-MINI-02, RevK:ESP32-PICO-MINI-02, symbol RevK:ESP32-PICO-MINI-02
Connections:
- net +3V3: now also J5.3 (3V3), U1.3 (3V3)
- net EN: now also C8.2, U1.8 (EN)
- net GND: now also C8.1, J5.1 (GND), U1.1 (GND), U1.11 (GND), U1.14 (GND), U1.2 (GND), U1.36 (GND), U1.37 (GND), U1.38 (GND), U1.39 (GND), U1.40 (GND), U1.41 (GND), U1.42 (GND), U1.43 (GND), U1.44 (GND), U1.45 (GND), U1.46 (GND), U1.47 (GND), U1.48 (GND), U1.49 (GND), U1.50 (GND), U1.51 (GND), U1.52 (GND), U1.53 (GND)
- net GPIO0: now also J5.2 (0), U1.23 (IO0)
- net I: now also J5.4 (Rx), U1.30 (RXD0)
- net O: now also J5.5 (Tx), U1.31 (TXD0)
- no-connect marks 12 -> 9

Commit message: PCB Update
Parts:
- C5: LCSC Part # C30926 -> (none); MPN (none) -> C30926
- C6: LCSC Part # C19110 -> (none); MPN (none) -> C19110
- C7: LCSC Part # C17024 -> (none); MPN (none) -> C17024
- D1: LCSC Part # C409798 -> (none); MPN (none) -> C409798
- D6: JLCPCB Rotation Offset 0 -> (none); LCSC Part # C143805 -> (none); MPN (none) -> C143805
- L1: LCSC Part # C354575 -> (none); MPN (none) -> C354575
- R11: LCSC Part # C14675 -> (none); MPN (none) -> C14675
- R12: LCSC Part # C100001 -> (none); MPN (none) -> C100001
- U1: LCSC Part # C2980306 -> (none); MPN (none) -> C2980306
- U3: JLCPCB Rotation Offset 90 -> (none); LCSC Part # C87080 -> (none); MPN (none) -> C87080
