File: PCB/Generic4/Generic4.kicad_pcb (KiCad board)
At the start: 2 copper layers, 13.2 x 19.5 mm, 19 parts, among them J1 Shelly, J2 SPOX, J3 Conn_01x05, U1 ESP32-PICO-MINI-02, U2 LMR16006+FB

Commit message: Started some updates, not all complete
Parts:
- removed C2: 0.1uF, RevK:Hidden
- removed C3: 2.2uF, RevK:Hidden
- removed C4: 10uF, RevK:Hidden
- removed D2: Schottky, RevK:Hidden
- removed L1: 6.8uH, RevK:Hidden
- removed R5: 100k 1% or 0R, RevK:R_0603
- removed R6: 30k 1% or NF, RevK:R_0603
- removed U2: LMR16006+FB, RevK:SOT-23-Thin-6-Reg
- added C6: 100nF, RevK:C_0603_, B.Cu at (101.8, 41.9)
- added C7: 2.2uF, RevK:C_0805_, B.Cu at (100.6, 45.1)
- added C8: 10uF, RevK:C_0805_, B.Cu at (94.3, 45.1)
- added D3: Schottky, RevK:D_1206_, B.Cu at (97.5, 44.8)
- added L2: 6.8uH, RevK:L_4x4_, B.Cu at (95.8, 41.6)
- added R7: 100k 1%, RevK:R_0603, B.Cu at (105.1, 39.4)
- added R8: 30k 1%, RevK:R_0603, B.Cu at (102.5, 39.4)
- added U3: LMR16006YDDCR, RevK:SOT-23-Thin-6-Reg, B.Cu at (99.8, 41.6)
- C1: value 10nF -> 1uF
Routing:
- net Net-(U3-FB): track 0.00 -> 3.95 mm
- net Net-(R5-Pad2): track 3.95 -> 0.00 mm
- net GND: track 40.8 -> 42.5 mm
Other:
- board text added: "22/19/7"
- board text removed: "RGB: 22/19/7"
