File: PCB/Generic4/Generic4.kicad_sch (KiCad schematic)
At the start: 19 parts, among them J1 Shelly, J2 SPOX, J3 Conn_01x05, U1 ESP32-PICO-MINI-02, U2 LMR16006+FB

Commit message: Started some updates, not all complete
Parts:
- removed C4: 10uF, RevK:Hidden, symbol RevK:Hidden
- removed R6: 30k 1% or NF, RevK:R_0603, symbol Device:R
- removed U2: LMR16006+FB, RevK:SOT-23-Thin-6-Reg, symbol RevK:LMR16006+FB
- added C1: 100nF, RevK:C_0603_, symbol RevK:Hidden
- added R4: 100k 1%, RevK:R_0603, symbol Device:R
- added U2: LMR16006YDDCR, RevK:SOT-23-Thin-6-Reg, symbol RevK:LMR16006XDDCR
- C1: value 10nF -> 1uF
- C2: value 0.1uF -> 2.2uF; footprint RevK:Hidden -> RevK:C_0805_; LCSC Part # (none) -> C19110; Note X7R or X5R 0603 -> (none)
- C3: value 2.2uF -> 10uF; footprint RevK:Hidden -> RevK:C_0805_; LCSC Part # (none) -> C17024; Note 0603 or 0805 -> (none)
- D2: footprint RevK:Hidden -> RevK:D_1206_; JLCPCB Rotation Offset (none) -> 0; LCSC Part # (none) -> C143805; Part No CD1206-B2100 -> (none)
- L1: footprint RevK:Hidden -> RevK:L_4x4_; LCSC Part # (none) -> C354575; Manufacturer Laird -> (none); Part No TYA4020 -> (none)
- R5: value 100k 1% or 0R -> 30k 1%; LCSC Part # (none) -> C100001
Connections:
- net +3.3V: now also R4.1, U2.7 (VOUT); no longer R5.1
- net DC: now also U2.4 (SHDN), U2.5 (VIN)
- net GND: now also R5.1, U2.2 (GND)
- net at R5.2: now also R4.2, U2.3 (FB)

Commit message: PCB Update
Parts:
- C6: renamed from C1; LCSC Part # C30926 -> (none); MPN (none) -> C30926
- C7: renamed from C2; LCSC Part # C19110 -> (none); MPN (none) -> C19110
- C8: renamed from C3; LCSC Part # C17024 -> (none); MPN (none) -> C17024
- D3: renamed from D2; JLCPCB Rotation Offset 0 -> (none); LCSC Part # C143805 -> (none); MPN (none) -> C143805
- L2: renamed from L1; LCSC Part # C354575 -> (none); MPN (none) -> C354575
- R7: renamed from R4; LCSC Part # C14675 -> (none); MPN (none) -> C14675
- R8: renamed from R5; LCSC Part # C100001 -> (none); MPN (none) -> C100001
- U3: renamed from U2; JLCPCB Rotation Offset 180 -> (none); LCSC Part # C290195 -> (none); MPN (none) -> C290195
