File: PCB/Generic6/Generic6.kicad_pcb (KiCad board)
At the start: 2 copper layers, 17.8 x 15.2 mm, 29 parts, among them J1 Shelly, P1 4, P10 37, P11 36, P12 DC, P2 32, P3 13, P4 25, P5 26, P6 33, P7 8, P8 27, P9 14, U1 ESP32-PICO-MINI-02, U2 LMR16006+FB

Commit message: Started some updates, not all complete
Parts:
- removed C2: 0.1uF, RevK:Hidden
- removed C3: 2.2uF, RevK:Hidden
- removed C4: 10uF, RevK:Hidden
- removed D2: Schottky, RevK:Hidden
- removed L1: 6.8uH, RevK:Hidden
- removed R5: 100k 1% or 0R, RevK:R_0402
- removed R6: 30k 1% or NF, RevK:R_0402
- removed U2: LMR16006+FB, RevK:RegulatorBlockFB
- added C6: 100nF, RevK:C_0603_, B.Cu at (77.5, 47.0)
- added C7: 2.2uF, RevK:C_0805_, B.Cu at (77.3, 42.2)
- added C8: 10uF, RevK:C_0805_, B.Cu at (77.3, 44.7)
- added D3: Schottky, RevK:D_1206_, B.Cu at (81.7, 51.4)
- added L2: 6.8uH, RevK:L_4x4_, B.Cu at (86.4, 52.6)
- added R7: 100k 1%, RevK:R_0603, B.Cu at (100.2, 38.8)
- added R8: 30k 1%, RevK:R_0603, B.Cu at (103.5, 38.8)
- added U3: LMR16006YDDCR, RevK:SOT-23-Thin-6-Reg, B.Cu at (100.5, 42.9)
- C1: value 10nF -> 1uF
- P10: value 37 -> 20
- P11: value 36 -> 15
Routing:
- net Net-(U3-FB): track 0.00 -> 8.10 mm
- net Net-(R5-Pad2): track 8.10 -> 0.00 mm
Other:
- board text added: "${CURRENT_DATE}"
- board text removed: "${DATE}"

Commit message: PCB Update
Parts:
- moved C6 25.4 mm to (102.6, 43.1), turned to 90 degrees
- moved C7 24.5 mm to (101.3, 46.5), turned to -90 degrees
- moved C8 17.9 mm to (95.1, 46.5), turned to -90 degrees
- moved D3 17.4 mm to (98.2, 46.1)
- moved L2 14.1 mm to (96.6, 42.9)
Connections:
- J1 pad 2: Net-(J1-0) -> unconnected-(J1-0-Pad2)
- J1 pad 4: Net-(J1-Rx) -> unconnected-(J1-Rx-Pad4)
- J1 pad 5: Net-(J1-Tx) -> unconnected-(J1-Tx-Pad5)
- U1 pad 1: GND -> Net-(U1-GND-Pad1)
- U1 pad 11: GND -> Net-(U1-GND-Pad1)
- U1 pad 14: GND -> Net-(U1-GND-Pad1)
- U1 pad 2: GND -> Net-(U1-GND-Pad1)
- U1 pad 23: Net-(J1-0) -> unconnected-(U1-IO0-Pad23)
- U1 pad 3: +3V3 -> unconnected-(U1-3V3-Pad3)
- U1 pad 30: Net-(J1-Rx) -> unconnected-(U1-RXD0-Pad30)
- U1 pad 31: Net-(J1-Tx) -> unconnected-(U1-TXD0-Pad31)
- U1 pad 36: GND -> Net-(U1-GND-Pad1)
- U1 pad 37: GND -> Net-(U1-GND-Pad1)
- U1 pad 38: GND -> Net-(U1-GND-Pad1)
- U1 pad 39: GND -> Net-(U1-GND-Pad1)
- U1 pad 40: GND -> Net-(U1-GND-Pad1)
- U1 pad 41: GND -> Net-(U1-GND-Pad1)
- U1 pad 42: GND -> Net-(U1-GND-Pad1)
- U1 pad 43: GND -> Net-(U1-GND-Pad1)
- U1 pad 44: GND -> Net-(U1-GND-Pad1)
- U1 pad 45: GND -> Net-(U1-GND-Pad1)
- U1 pad 46: GND -> Net-(U1-GND-Pad1)
- U1 pad 47: GND -> Net-(U1-GND-Pad1)
- U1 pad 48: GND -> Net-(U1-GND-Pad1)
- U1 pad 49: GND -> Net-(U1-GND-Pad1)
- U1 pad 50: GND -> Net-(U1-GND-Pad1)
- U1 pad 51: GND -> Net-(U1-GND-Pad1)
- U1 pad 52: GND -> Net-(U1-GND-Pad1)
- U1 pad 53: GND -> Net-(U1-GND-Pad1)
Routing:
- net (no net): track 0.00 -> 9.70 mm, vias 0 -> 1
- net Net-(J1-0): track 4.80 -> 0.00 mm, vias 1 -> 0
- net Net-(J1-Tx): track 3.04 -> 0.00 mm
- net Net-(J1-Rx): track 1.86 -> 0.00 mm
- net GND: track 30.2 -> 29.4 mm, vias 18 -> 17
- net Net-(U1-GND-Pad1): track 0.00 -> 0.86 mm, vias 0 -> 1
