File: PCB/Generic6/Generic6.kicad_sch (KiCad schematic)
At the start: 29 parts, among them J1 Shelly, P1 4, P10 20, P11 15, P12 DC, P2 32, P3 13, P4 25, P5 26, P6 33, P7 8, P8 27, P9 14, U1 ESP32-PICO-MINI-02, U2 LMR16006+FB

Commit message: Started some updates, not all complete
Parts:
- removed C4: 10uF, RevK:Hidden, symbol RevK:Hidden
- removed R6: 30k 1% or NF, RevK:R_0402, symbol Device:R
- removed U2: LMR16006+FB, RevK:RegulatorBlockFB, symbol RevK:LMR16006+FB
- added C1: 100nF, RevK:C_0603_, symbol RevK:Hidden
- added R4: 100k 1%, RevK:R_0603, symbol Device:R
- added U2: LMR16006YDDCR, RevK:SOT-23-Thin-6-Reg, symbol RevK:LMR16006XDDCR
- C1: value 10nF -> 1uF
- C2: value 0.1uF -> 2.2uF; footprint RevK:Hidden -> RevK:C_0805_; LCSC Part # (none) -> C19110; Note X7R or X5R 0603 -> (none)
- C3: value 2.2uF -> 10uF; footprint RevK:Hidden -> RevK:C_0805_; LCSC Part # (none) -> C17024; Note 0603 or 0805 -> (none)
- D2: footprint RevK:Hidden -> RevK:D_1206_; JLCPCB Rotation Offset (none) -> 0; LCSC Part # (none) -> C143805; Part No CD1206-B2100 -> (none)
- L1: footprint RevK:Hidden -> RevK:L_4x4_; LCSC Part # (none) -> C354575; Manufacturer Laird -> (none); Part No TYA4020 -> (none)
- R5: value 100k 1% or 0R -> 30k 1%; footprint RevK:R_0402 -> RevK:R_0603; LCSC Part # (none) -> C100001
Connections:
- net +3V3: now also R4.1, U2.7 (VOUT); no longer R5.1
- net GND: now also R5.1, U2.2 (GND)
- net at P12.1 (P): now also U2.4 (SHDN), U2.5 (VIN)
- net at J1.2 (0): now also U1.23 (IO0)
- net at U1.23 (IO0): no longer J1.2 (0)
- net at J1.4 (Rx): now also U1.30 (RXD0)
- net at J1.5 (Tx): now also U1.31 (TXD0)
- net at R5.2: now also R4.2, U2.3 (FB)
- new net: J1.1 (GND), U1.1 (GND)
- new net: J1.3 (3V3), U1.3 (3V3)

Commit message: PCB Update
Parts:
- C6: renamed from C1; LCSC Part # C30926 -> (none); MPN (none) -> C30926
- C7: renamed from C2; LCSC Part # C19110 -> (none); MPN (none) -> C19110
- C8: renamed from C3; LCSC Part # C17024 -> (none); MPN (none) -> C17024
- D3: renamed from D2; JLCPCB Rotation Offset 0 -> (none); LCSC Part # C143805 -> (none); MPN (none) -> C143805
- L2: renamed from L1; LCSC Part # C354575 -> (none); MPN (none) -> C354575
- R7: renamed from R4; LCSC Part # C14675 -> (none); MPN (none) -> C14675
- R8: renamed from R5; LCSC Part # C100001 -> (none); MPN (none) -> C100001
- U1: MPN (none) -> C2980306
- U3: renamed from U2; JLCPCB Rotation Offset 180 -> (none); LCSC Part # C290195 -> (none); MPN (none) -> C290195
Connections:
- net +3V3: no longer U1.3 (3V3)
- net GND: no longer U1.1 (GND), U1.11 (GND), U1.14 (GND), U1.2 (GND), U1.36 (GND), U1.37 (GND), U1.38 (GND), U1.39 (GND), U1.40 (GND), U1.41 (GND), U1.42 (GND), U1.43 (GND), U1.44 (GND), U1.45 (GND), U1.46 (GND), U1.47 (GND), U1.48 (GND), U1.49 (GND), U1.50 (GND), U1.51 (GND), U1.52 (GND), U1.53 (GND)
- net at U1.1 (GND): now also U1.11 (GND), U1.14 (GND), U1.2 (GND), U1.36 (GND), U1.37 (GND), U1.38 (GND), U1.39 (GND), U1.40 (GND), U1.41 (GND), U1.42 (GND), U1.43 (GND), U1.44 (GND), U1.45 (GND), U1.46 (GND), U1.47 (GND), U1.48 (GND), U1.49 (GND), U1.50 (GND), U1.51 (GND), U1.52 (GND), U1.53 (GND); no longer J1.1 (GND)
- net at U1.23 (IO0): no longer J1.2 (0)
- net at U1.3 (3V3): no longer J1.3 (3V3)
- net at U1.30 (RXD0): no longer J1.4 (Rx)
- net at U1.31 (TXD0): no longer J1.5 (Tx)
