File: PCB/USBC/USBC.kicad_sch (KiCad schematic)
At the start: 29 parts, among them J1 USB-C-Plug-V, J2 Shelly, J3 USB-PROG, J4 Conn_01x03_Socket, U2 ESP32-S3-MINI-1, U5 MD8942, U8 VEML6040

Commit message: More solid plug
Parts:
- J1: LCSC Part # C283539 -> C399938
Changed lines of the file:
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@@
       (effects (font (size 1.27 1.27)) hide)
     )
-    (property "LCSC Part #" "C283539" (at 243.84 65.405 0)
+    (property "LCSC Part #" "C399938" (at 243.84 65.405 0)
       (effects (font (size 1.27 1.27)) hide)
     )

Commit message: Fix CC
Parts:
- R2: value 56K -> 5K1
Connections:
- net GND: now also R2.2
- net VBUS: no longer R2.2
Other:
- note added: "Yes, NC as this is a plug"
Changed lines of the file:
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@@
     (stroke (width 0) (type default))
+  )
+  (text "Yes, NC as this is a plug" (at 255.905 60.325 0)
+    (effects (font (size 1.27 1.27)) (justify left bottom))
   )
   (global_label "D+" (shape bidirectional) (at 259.08 67.945 0) (fields_autoplaced)
@@
     (property "Intersheetrefs" "${INTERSHEET_REFS}" (at 154.8232 72.3106 0)
       (effects (font (size 1.27 1.27)) (justify right) hide)
-    )
-  )
-  (global_label "VBUS" (shape output) (at 266.7 55.245 0) (fields_autoplaced)
-    (effects (font (size 1.27 1.27)) (justify left))
-    (property "Intersheetrefs" "${INTERSHEET_REFS}" (at 273.8502 55.245 0)
-      (effects (font (size 1.27 1.27)) (justify left) hide)
     )
   )
@@
       (effects (font (size 1.27 1.27)))
     )
-    (property "Value" "56K" (at 262.89 55.245 90)
+    (property "Value" "5K1" (at 262.89 55.245 90)
       (effects (font (size 1.27 1.27)))
     )
@@
         )
       )
+    )
+  )
+  (symbol (lib_name "GND_2") (lib_id "power:GND") (at 266.7 55.245 90) (unit 1)
+    (in_bom yes) (on_board yes) (dnp no) (fields_autoplaced)
+    (property "Reference" "#PWR06" (at 273.05 55.245 0)
+      (effects (font (size 1.27 1.27)) hide)
+    )
+    (property "Value" "GND" (at 269.875 55.245 90)
+      (effects (font (size 1.27 1.27)) (justify right))
+    )
+    (property "Footprint" "" (at 266.7 55.245 0)
+      (effects (font (size 1.27 1.27)) hide)
+    )
+    (property "Datasheet" "" (at 266.7 55.245 0)
+      (effects (font (size 1.27 1.27)) hide)
+    )
+    (pin "1")
+    (instances
+      (project "USBC"
+        (path "/2d210a96-f81f-42a9-8bf4-1b43c11086f3"
+          (reference "#PWR06") (unit 1)
+        )
+      )

Commit message: Adjusted
Parts:
- J1: JLCPCB Rotation Offset 90 -> (none)
Changed lines of the file:
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@@
-      (effects (font (size 1.27 1.27)) hide)
-    )
-    (property "JLCPCB Rotation Offset" "90" (at 243.84 45.9049 0)
       (effects (font (size 1.27 1.27)) hide)
     )

Commit message: Tweak
Parts:
- added D6, D7: XL-1010RGBC-WS2812B, RevK:SMD1010, symbol RevK:WS2812B-1mm
Connections:
- net GND: now also D6.3 (-), D7.3 (-)
- net VBUS: now also D6.2 (+), D7.2 (+)
- net at D5.1 (O): now also D6.4 (I); no longer J4.2 (Pin_2)
- new net: D7.1 (O), J4.2 (Pin_2)
- new net: D6.1 (O), D7.4 (I)
- no-connect marks 25 -> 23
Other:
- moved on the sheet: C3, C4, J4, R1

Commit message: Tweak layout
Parts:
- C6: value 10uF 50V -> 10uF 35V; LCSC Part # C1591 -> C194427
Changed lines of the file:
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@@
       (effects (font (size 1.27 1.27)) (justify left))
     )
-    (property "Value" "10uF 50V" (at 200.025 121.92 0)
+    (property "Value" "10uF 35V" (at 200.025 121.92 0)
       (effects (font (size 1.27 1.27)) (justify left))
     )
@@
       (effects (font (size 1.27 1.27)) hide)
     )
-    (property "LCSC Part #" "C1591" (at 193.675 121.92 0)
+    (property "LCSC Part #" "C194427" (at 193.675 121.92 0)
       (effects (font (size 1.27 1.27)) hide)
     )

Commit message: PCB Update
Parts:
- C6: LCSC Part # C194427 -> (none); MPN (none) -> C194427
- C7: LCSC Part # C1691 -> (none); MPN (none) -> C1691
- D1, D2, D3, D4, D5, D6, D7: LCSC Part # C5349953 -> (none); MPN (none) -> C5349953
- J1: LCSC Part # C399938 -> (none); MPN (none) -> C399938
- U1: renamed from U8; JLCPCB Rotation Offset 90 -> (none); LCSC Part # C78465 -> (none); MPN (none) -> C78465
- U2: LCSC Part # C3013941 -> (none); MPN (none) -> C3013941
- U5: LCSC Part # C2684786 -> (none); MPN (none) -> C2684786
