File: PCB/GenericS3Bat/GenericS3.kicad_pcb (KiCad board)
At the start: 2 copper layers, 70 x 70 mm, 73 parts, among them J1 USB-C-Socket-V, J2 JST-PH-SM4-TB, P1 33, P10 42, P11 45, P12 46, P13 47, P14 48, P15 18, P16 19, P17 14, P18 15, P19 16, P2 34, P20 17, P21 6, P22 7, P23 8, P24 9, P25 20, P26 10, P27 11, P28 12, P29 13, P3 35, P30 1, P31 2, P32 3, P33 4, P34 5, P35 21, P36 43, P37 44, P38 0, P39 ⏚, P4 36, P40 ⏚, P41 ⏚, P42 ⏚, P43 +, P44 +, P45 +, P46 +, P5 37, P6 38, P7 39, P8 40, P9 41, Q1 CJ2301, SW1 SW_Push_DPDT, U1 ESP32-S3-MINI-1, U2 TP4054, U4 ME6211C33M5G-N

Commit message: Change reg
Parts:
- moved J1 0.50 mm to (119.0, 91.0)
Routing:
- net GND: track 17.4 -> 14.8 mm
